File: appendix_TMC2660_X.sch (KiCad schematic (older format))
At the start: 13 parts

Commit message: added FTDI chip
Parts:
- added J?: Conn_01x06, symbol Connector_Generic:Conn_01x06
- added J?: Conn_01x04, symbol Connector_Generic:Conn_01x04
Connections:
- wire segments 94 -> 102

Commit message: merged hierarchical schematics
Parts:
- removed J?: Conn_01x06, symbol Connector_Generic:Conn_01x06
