File: appendix_TMC2660_X.sch (KiCad schematic (older format))
At the start: 14 parts

Commit message: pre Annotation 1
Parts:
- added C? (x12): 100n, symbol Device:C
- added C? (x3): 470n, symbol Device:C
- added C? (x3): 220n, symbol Device:C
- added C? (x6): 10u, symbol Device:C
- added J? (x3): Conn_01x04, symbol Connector_Generic:Conn_01x04
- added R? (x6): 10R, symbol Device:R
- added R? (x6): 0R1, symbol Device:R
- added U? (x3): TMC2660, symbol FHNW-Pro4E-FS19T8-Library:TMC2660
Connections:
- net labels added: D_TMC_CS_E1, D_TMC_CS_Y, D_TMC_CS_Z1, D_TMC_DIR_E1, D_TMC_DIR_Y, D_TMC_DIR_Z1, D_TMC_EN_E1, D_TMC_EN_Y, D_TMC_EN_Z1, D_TMC_STEP_E1, D_TMC_STEP_Y, D_TMC_STEP_Z1, MOT_E1_A1, MOT_E1_A2, MOT_E1_B1, MOT_E1_B2, MOT_X_A1, MOT_X_A2, MOT_X_B1, MOT_X_B2, MOT_Y_A1, MOT_Y_A2, MOT_Y_B1, MOT_Y_B2, MOT_Z1_A1, MOT_Z1_A2, MOT_Z1_B1, MOT_Z1_B2
- wire segments 102 -> 348
Other:
- note added: "EXTRUDER 1"
- note added: "X AXIS"
- note added: "Y AXIS"
- note added: "Z AXIS 1"
- moved on the sheet: C?, J?, R?, U?

Commit message: 1st annotation, footprints, netlist
Parts:
- C601, C602, C603, C604, C605, C606, C607, C608, C609, C610, C611, C612, C613, C614, C615, C616, C617, C618, C619, C620, C621, C622, C623, C624, C625, C626, C627, C628, C629, C630, C631, C632: renamed from C?; footprint (none) -> Capacitors_SMD:C_0805
- J601, J602, J603, J604: renamed from J?; footprint (none) -> Connector_PinHeader_2.54mm:PinHeader_1x04_P2.54mm_Vertical
- R601, R602, R603, R604, R605, R606, R607, R608, R609, R610, R611, R612, R613, R614, R615, R616: renamed from R?; footprint (none) -> Resistors_SMD:R_0805
- U601, U602, U603, U604: renamed from U?; footprint (none) -> digikey-footprints:TQFP-44_10x10mm
