File: FHNW-Pro4E-FS19T8-3DPrinterBoard-STM32.sch (KiCad schematic (older format))
At the start: 6 parts, among them U101 LM2675M-3.3

Commit message: started layouting TMC2660
Parts:
- C101, C102, C103: footprint Capacitors_SMD:C_0805 -> Capacitors_SMD:C_0603
Connections:
- no-connect marks 0 -> 1
Other:
- note removed: "duplicate for Y, Z, E\nafter X is finished \n(connectors from Tobi are missing)"
- moved on the sheet: C101, C102, C103, D101, L101, U101
Changed lines of the file:
@@
 $EndDescr
 $Sheet
-S 4300 1000 2500 1800
+S 3200 1000 1750 1650
 U 5CA3954A
 F0 "appendix_STM32F103" 50
@@
 $EndSheet
 $Sheet
-S 4300 3200 2500 600
+S 3200 3150 1750 1650
 U 5CA395A8
 F0 "appendix_ESP32" 50
@@
 $EndSheet
 $Sheet
-S 1050 2500 1250 900
+S 5400 2050 1150 600
 U 5CA39F21
 F0 "appendix_SENSORS_POWER" 50
@@
 $EndSheet
 $Sheet
-S 7100 2700 1150 650
+S 1000 1000 1150 650
 U 5CA3CC17
 F0 "appendix_UART_USB" 50
@@
 $EndSheet
 $Sheet
-S 9800 900  1200 750
+S 5400 1000 1150 750
 U 5CA3FF44
 F0 "appendix_TMC2660_X" 50
 F1 "appendix_TMC2660_X.sch" 50
 $EndSheet
-Text Notes 8400 1250 0    50   ~ 0
-duplicate for Y, Z, E\nafter X is finished \n(connectors from Tobi are missing)
 $Bitmap
-Pos 5600 3500
+Pos 4100 3650
 Scale 1.000000
 Data
@@
 $EndBitmap
 $Bitmap
-Pos 5550 1900
+Pos 4050 1450
 Scale 1.000000
 Data
@@
 $EndBitmap
 $Bitmap
-Pos 10400 1300
+Pos 5950 1400
 Scale 1.000000
 Data
@@
 $EndBitmap
 $Bitmap
-Pos 7650 3000
+Pos 1350 1200
 Scale 1.000000
 Data
@@
 EndData
 $EndBitmap
-Text Notes 1350 5750 0    50   ~ 0
+Text Notes 2400 5900 0    50   ~ 0
 what about on/#off input?\n
 $Comp
 L Regulator_Switching:LM2675M-3.3 U101
 U 1 1 5CA6A12A
-P 1850 6500
-F 0 "U101" H 1850 6967 50  0000 C CNN
-F 1 "LM2675M-3.3" H 1850 6876 50  0000 C CNN
-F 2 "Housings_SOIC:SOIC-8-1EP_3.9x4.9mm_Pitch1.27mm" H 1900 6150 50  0001 L CIN
-F 3 "http://www.ti.com/lit/ds/symlink/lm2675.pdf" H 1850 6500 50  0001 C CNN
-	1    1850 6500
+P 2900 6650
+F 0 "U101" H 2900 7117 50  0000 C CNN
+F 1 "LM2675M-3.3" H 2900 7026 50  0000 C CNN
+F 2 "Housings_SOIC:SOIC-8-1EP_3.9x4.9mm_Pitch1.27mm" H 2950 6300 50  0001 L CIN
+F 3 "http://www.ti.com/lit/ds/symlink/lm2675.pdf" H 2900 6650 50  0001 C CNN
+	1    2900 6650
 	1    0    0    -1
 $EndComp
 Wire Wire Line
-	2000 7100 1850 7100
+	3050 7250 2900 7250
 $Comp
 L Device:D_Schottky D101
 U 1 1 5CA6A134
-P 2150 7100
-F 0 "D101" H 2150 7000 50  0000 C CNN
-F 1 "Shottky STPS1L30A" H 2150 7200 50  0000 C CNN
-F 2 "Diodes_SMD:D_1206" H 2150 7100 50  0001 C CNN
-F 3 "~" H 2150 7100 50  0001 C CNN
-	1    2150 7100
+P 3200 7250
+F 0 "D101" H 3200 7150 50  0000 C CNN
+F 1 "Shottky STPS1L30A" H 3200 7350 50  0000 C CNN
+F 2 "Diodes_SMD:D_1206" H 3200 7250 50  0001 C CNN
+F 3 "~" H 3200 7250 50  0001 C CNN
+	1    3200 7250
 	-1   0    0    1
 $EndComp
@@
 L power:+3.3V #PWR0101
 U 1 1 5CA6A13E
-P 3900 6150
-F 0 "#PWR0101" H 3900 6000 50  0001 C CNN
-F 1 "+3.3V" H 3915 6323 50  0000 C CNN
-F 2 "" H 3900 6150 50  0001 C CNN
-F 3 "" H 3900 6150 50  0001 C CNN
-	1    3900 6150
+P 4950 6300
+F 0 "#PWR0101" H 4950 6150 50  0001 C CNN
+F 1 "+3.3V" H 4965 6473 50  0000 C CNN
+F 2 "" H 4950 6300 50  0001 C CNN
+F 3 "" H 4950 6300 50  0001 C CNN
+	1    4950 6300
 	1    0    0    -1
 $EndComp
 Wire Wire Line
-	1850 6900 1850 7100
+	2900 7050 2900 7250
 $Comp
 L power:GND #PWR0102
 U 1 1 5CA6A14E
-P 3900 7250
-F 0 "#PWR0102" H 3900 7000 50  0001 C CNN
-F 1 "GND" H 3905 7077 50  0000 C CNN
-F 2 "" H 3900 7250 50  0001 C CNN
-F 3 "" H 3900 7250 50  0001 C CNN
-	1    3900 7250
+P 4950 7400
+F 0 "#PWR0102" H 4950 7150 50  0001 C CNN
+F 1 "GND" H 4955 7227 50  0000 C CNN
+F 2 "" H 4950 7400 50  0001 C CNN
+F 3 "" H 4950 7400 50  0001 C CNN
+	1    4950 7400
 	1    0    0    -1
 $EndComp
@@
 L power:+12V #PWR0103
 U 1 1 5CA6A160
-P 1150 6150
-F 0 "#PWR0103" H 1150 6000 50  0001 C CNN
-F 1 "+12V" H 1165 6323 50  0000 C CNN
-F 2 "" H 1150 6150 50  0001 C CNN
-F 3 "" H 1150 6150 50  0001 C CNN
-	1    1150 6150
+P 2200 6300
+F 0 "#PWR0103" H 2200 6150 50  0001 C CNN
+F 1 "+12V" H 2215 6473 50  0000 C CNN
+F 2 "" H 2200 6300 50  0001 C CNN
+F 3 "" H 2200 6300 50  0001 C CNN
+	1    2200 6300
 	1    0    0    -1
 $EndComp
@@
 L power:GND #PWR0104
 U 1 1 5CA6A166
-P 1150 7250
-F 0 "#PWR0104" H 1150 7000 50  0001 C CNN
-F 1 "GND" H 1155 7077 50  0000 C CNN
-F 2 "" H 1150 7250 50  0001 C CNN
-F 3 "" H 1150 7250 50  0001 C CNN
-	1    1150 7250
+P 2200 7400
+F 0 "#PWR0104" H 2200 7150 50  0001 C CNN
+F 1 "GND" H 2205 7227 50  0000 C CNN
+F 2 "" H 2200 7400 50  0001 C CNN
+F 3 "" H 2200 7400 50  0001 C CNN
+	1    2200 7400
 	1    0    0    -1
 $EndComp
@@
 L Device:CP C101
 U 1 1 5CA6A16C
-P 3900 6500
-F 0 "C101" H 4018 6546 50  0000 L CNN
-F 1 "100uF" H 4018 6455 50  0000 L CNN
-F 2 "Capacitors_SMD:C_0805" H 3938 6350 50  0001 C CNN
-F 3 "~" H 3900 6500 50  0001 C CNN
-	1    3900 6500
+P 4950 6650
+F 0 "C101" H 5068 6696 50  0000 L CNN
+F 1 "100uF" H 5068 6605 50  0000 L CNN
+F 2 "Capacitors_SMD:C_0603" H 4988 6500 50  0001 C CNN
+F 3 "~" H 4950 6650 50  0001 C CNN
+	1    4950 6650
 	1    0    0    -1
 $EndComp
@@
 L Device:L L101
 U 1 1 5CA6A172
-P 3100 6750
-F 0 "L101" H 3059 6704 50  0000 R CNN
-F 1 "47uH DO3316-473" H 3059 6795 50  0000 R CNN
-F 2 "Inductors_SMD:L_10.4x10.4_H4.8" H 3100 6750 50  0001 C CNN
-F 3 "~" H 3100 6750 50  0001 C CNN
-	1    3100 6750
+P 4150 6900
+F 0 "L101" H 4109 6854 50  0000 R CNN
+F 1 "47uH DO3316-473" H 4109 6945 50  0000 R CNN
+F 2 "Inductors_SMD:L_10.4x10.4_H4.8" H 4150 6900 50  0001 C CNN
+F 3 "~" H 4150 6900 50  0001 C CNN
+	1    4150 6900
 	-1   0    0    1
 $EndComp
@@
 L Device:CP C102
 U 1 1 5CA6A178
-P 1150 6600
-F 0 "C102" H 800 6750 50  0000 L CNN
-F 1 "330uF" H 800 6450 50  0000 L CNN
-F 2 "Capacitors_SMD:C_0805" H 1188 6450 50  0001 C CNN
-F 3 "~" H 1150 6600 50  0001 C CNN
-	1    1150 6600
+P 2200 6750
+F 0 "C102" H 1850 6900 50  0000 L CNN
+F 1 "330uF" H 1850 6600 50  0000 L CNN
+F 2 "Capacitors_SMD:C_0603" H 2238 6600 50  0001 C CNN
+F 3 "~" H 2200 6750 50  0001 C CNN
+	1    2200 6750
 	1    0    0    -1
 $EndComp
@@
 L Device:C C103
 U 1 1 5CA6A17E
-P 2550 6750
-F 0 "C103" H 2665 6796 50  0000 L CNN
-F 1 "0.01uF/50V" H 2600 6650 50  0000 L CNN
-F 2 "Capacitors_SMD:C_0805" H 2588 6600 50  0001 C CNN
-F 3 "~" H 2550 6750 50  0001 C CNN
-	1    2550 6750
+P 3600 6900
+F 0 "C103" H 3715 6946 50  0000 L CNN
+F 1 "0.01uF/50V" H 3650 6800 50  0000 L CNN
+F 2 "Capacitors_SMD:C_0603" H 3638 6750 50  0001 C CNN
+F 3 "~" H 3600 6900 50  0001 C CNN
+	1    3600 6900
 	1    0    0    -1
 $EndComp
 Wire Wire Line
-	1150 6150 1150 6300
+	2200 6300 2200 6450
 Wire Wire Line
-	1150 6750 1150 7100
+	2200 6900 2200 7250
 Wire Wire Line
-	1350 6300 1150 6300
-Connection ~ 1150 6300
+	2400 6450 2200 6450
+Connection ~ 2200 6450
 Wire Wire Line
-	1150 6300 1150 6450
+	2200 6450 2200 6600
 Wire Wire Line
-	1850 7100 1150 7100
-Connection ~ 1850 7100
-Connection ~ 1150 7100
+	2900 7250 2200 7250
+Connection ~ 2900 7250
+Connection ~ 2200 7250
 Wire Wire Line
-	1150 7100 1150 7250
+	2200 7250 2200 7400
 Wire Wire Line
-	2300 7100 2400 7100
+	3350 7250 3450 7250
 Wire Wire Line
-	2350 6700 2400 6700
+	3400 6850 3450 6850
 Wire Wire Line
-	2400 6700 2400 7100
-Connection ~ 2400 7100
+	3450 6850 3450 7250
+Connection ~ 3450 7250
 Wire Wire Line
-	2400 7100 2550 7100
+	3450 7250 3600 7250
 Wire Wire Line
-	2550 6600 2550 6500
+	3600 6750 3600 6650
 Wire Wire Line
-	2550 6500 2350 6500
+	3600 6650 3400 6650
 Wire Wire Line
-	2550 6900 2550 7100
-Connection ~ 2550 7100
+	3600 7050 3600 7250
+Connection ~ 3600 7250
 Wire Wire Line
-	2550 7100 3100 7100
+	3600 7250 4150 7250
 Wire Wire Line
-	3100 6900 3100 7100
+	4150 7050 4150 7250
 Wire Wire Line
-	3100 6600 3100 6300
+	4150 6750 4150 6450
 Wire Wire Line
-	3100 6300 2350 6300
+	4150 6450 3400 6450
 Wire Wire Line
-	3900 6350 3900 6300
+	4950 6500 4950 6450
 Wire Wire Line
-	3100 6300 3900 6300
-Connection ~ 3100 6300
-Connection ~ 3900 6300
+	4150 6450 4950 6450
+Connection ~ 4150 6450
+Connection ~ 4950 6450
 Wire Wire Line
-	3900 6300 3900 6150
+	4950 6450 4950 6300
 Wire Wire Line
-	3900 6650 3900 7250
+	4950 6800 4950 7400
+Wire Notes Line
+	2200 1200 3150 1200
+Wire Notes Line
+	2200 1500 2650 1500
+Wire Notes Line
+	2650 1500 2650 3350
+Wire Notes Line
+	2650 3350 3150 3350
+Wire Notes Line
+	5000 1250 5350 1250
+Wire Notes Line
+	5000 2300 5350 2300
+NoConn ~ 2400 6650
 $EndSCHEMATC

Commit message: Layout: all TMC / Schematic: Oli's comments
Parts:
- added F101: Fuse, symbol Device:Fuse
- added J101: Screw_Terminal_01x02, Connectors_Terminal_Blocks:TerminalBlock_Altech_AK300-2_P5.00mm, symbol Connector:Screw_Terminal_01x02
Connections:
- net labels added: +24V
- net labels removed: +12V
- wire segments 23 -> 28
Other:
- note removed: "what about on/#off input?\n"
Changed lines of the file:
@@
 EndData
 $EndBitmap
-Text Notes 2400 5900 0    50   ~ 0
-what about on/#off input?\n
 $Comp
 L Regulator_Switching:LM2675M-3.3 U101
@@
 $EndComp
 $Comp
-L power:+12V #PWR0103
-U 1 1 5CA6A160
-P 2200 6300
-F 0 "#PWR0103" H 2200 6150 50  0001 C CNN
-F 1 "+12V" H 2215 6473 50  0000 C CNN
-F 2 "" H 2200 6300 50  0001 C CNN
-F 3 "" H 2200 6300 50  0001 C CNN
-	1    2200 6300
-	1    0    0    -1
-$EndComp
-$Comp
 L power:GND #PWR0104
 U 1 1 5CA6A166
@@
 	5000 2300 5350 2300
 NoConn ~ 2400 6650
+$Comp
+L power:+24V #PWR?
+U 1 1 5CD67EF2
+P 2200 6300
+AR Path="/5CA3FF44/5CD67EF2" Ref="#PWR?"  Part="1"
+AR Path="/5CD67EF2" Ref="#PWR0103"  Part="1"
+F 0 "#PWR0103" H 2200 6150 50  0001 C CNN
+F 1 "+24V" H 2215 6473 50  0000 C CNN
+F 2 "" H 2200 6300 50  0001 C CNN
+F 3 "" H 2200 6300 50  0001 C CNN
+	1    2200 6300
+	1    0    0    -1
+$EndComp
+$Comp
+L Connector:Screw_Terminal_01x02 J101
+U 1 1 5CD68AD6
+P 1250 6450
+F 0 "J101" H 1400 6600 50  0000 C CNN
+F 1 "Screw_Terminal_01x02" H 1500 6200 50  0000 C CNN
+F 2 "Connectors_Terminal_Blocks:TerminalBlock_Altech_AK300-2_P5.00mm" H 1250 6450 50  0001 C CNN
+F 3 "~" H 1250 6450 50  0001 C CNN
+	1    1250 6450
+	-1   0    0    -1
+$EndComp
+$Comp
+L Device:Fuse F?
+U 1 1 5CE8417C
+P 1750 6450
+AR Path="/5CA39F21/5CE8417C" Ref="F?"  Part="1"
+AR Path="/5CE8417C" Ref="F101"  Part="1"
+F 0 "F101" V 1553 6450 50  0000 C CNN
+F 1 "Fuse" V 1644 6450 50  0000 C CNN
+F 2 "" V 1680 6450 50  0001 C CNN
+F 3 "~" H 1750 6450 50  0001 C CNN
+	1    1750 6450
+	0    1    1    0
+$EndComp
+Wire Wire Line
+	1450 6450 1600 6450
+Wire Wire Line
+	1900 6450 2200 6450
+Wire Wire Line
+	2200 7250 1600 7250
+Wire Wire Line
+	1600 7250 1600 6550
+Wire Wire Line
+	1600 6550 1450 6550
 $EndSCHEMATC
