File: FHNW-Pro4E-FS19T8-3DPrinterBoard-STM32.sch (KiCad schematic (older format))
At the start: 34 parts, among them J101 Screw_Terminal_01x02, T101 BUK963R3-60E, U101 LM2675M-3.3, U102 LM2675M-5

Commit message: Added comments to the schematic. Changed various component values (annotated only).
Parts:
- C101, C102, C107, C108: symbol Device:CP -> FHNW-Pro4E-FS19T8-3DPrinterBoard-STM32-rescue:CP-Device
- C103, C104, C106, C109: symbol Device:C -> FHNW-Pro4E-FS19T8-3DPrinterBoard-STM32-rescue:C-Device
- D101, D103: symbol Device:D_Schottky -> FHNW-Pro4E-FS19T8-3DPrinterBoard-STM32-rescue:D_Schottky-Device
- D102, D104: symbol Device:LED -> FHNW-Pro4E-FS19T8-3DPrinterBoard-STM32-rescue:LED-Device
- D105: symbol Device:D_Zener -> FHNW-Pro4E-FS19T8-3DPrinterBoard-STM32-rescue:D_Zener-Device
- F101: symbol Device:Fuse -> FHNW-Pro4E-FS19T8-3DPrinterBoard-STM32-rescue:Fuse-Device
- FB101, FB102: symbol Device:Ferrite_Bead_Small -> FHNW-Pro4E-FS19T8-3DPrinterBoard-STM32-rescue:Ferrite_Bead_Small-Device
- H101, H102, H103, H104: symbol Mechanical:MountingHole -> FHNW-Pro4E-FS19T8-3DPrinterBoard-STM32-rescue:MountingHole-Mechanical
- J101: symbol Connector:Screw_Terminal_01x02 -> FHNW-Pro4E-FS19T8-3DPrinterBoard-STM32-rescue:Screw_Terminal_01x02-Connector
- L101, L102: symbol Device:L -> FHNW-Pro4E-FS19T8-3DPrinterBoard-STM32-rescue:L-Device
- LOGO101: symbol SparkFun-Aesthetics:OSHW-LOGOM-COPPER -> FHNW-Pro4E-FS19T8-3DPrinterBoard-STM32-rescue:OSHW-LOGOM-COPPER-SparkFun-Aesthetics
- R101, R102, R103, R104: symbol Device:R -> FHNW-Pro4E-FS19T8-3DPrinterBoard-STM32-rescue:R-Device
- U101: symbol Regulator_Switching:LM2675M-3.3 -> FHNW-Pro4E-FS19T8-3DPrinterBoard-STM32-rescue:LM2675M-3.3-Regulator_Switching
- U102: symbol Regulator_Switching:LM2675M-5 -> FHNW-Pro4E-FS19T8-3DPrinterBoard-STM32-rescue:LM2675M-5-Regulator_Switching
Other:
- note added: "20A"
- note added: "C104 misplaced on the PCB,\nshould be near +3.3VA"
- note added: "GREEN"
Changed lines of the file:
@@
 	3800 7250 3650 7250
 $Comp
-L Device:D_Schottky D101
+L FHNW-Pro4E-FS19T8-3DPrinterBoard-STM32-rescue:D_Schottky-Device D101
 U 1 1 5CA6A134
 P 3950 7250
@@
 $EndComp
 $Comp
-L power:+3.3V #PWR0101
+L FHNW-Pro4E-FS19T8-3DPrinterBoard-STM32-rescue:+3.3V-power #PWR0101
 U 1 1 5CA6A13E
 P 5700 6300
@@
 	3650 7050 3650 7250
 $Comp
-L power:GND #PWR0102
+L FHNW-Pro4E-FS19T8-3DPrinterBoard-STM32-rescue:GND-power #PWR0102
 U 1 1 5CA6A14E
 P 5700 7400
@@
 $EndComp
 $Comp
-L power:GND #PWR0104
+L FHNW-Pro4E-FS19T8-3DPrinterBoard-STM32-rescue:GND-power #PWR0104
 U 1 1 5CA6A166
 P 2950 7400
@@
 $EndComp
 $Comp
-L Device:CP C101
+L FHNW-Pro4E-FS19T8-3DPrinterBoard-STM32-rescue:CP-Device C101
 U 1 1 5CA6A16C
 P 5700 6650
@@
 $EndComp
 $Comp
-L Device:L L101
+L FHNW-Pro4E-FS19T8-3DPrinterBoard-STM32-rescue:L-Device L101
 U 1 1 5CA6A172
 P 4900 6900
@@
 $EndComp
 $Comp
-L Device:CP C102
+L FHNW-Pro4E-FS19T8-3DPrinterBoard-STM32-rescue:CP-Device C102
 U 1 1 5CA6A178
 P 2950 6750
@@
 $EndComp
 $Comp
-L Device:C C103
+L FHNW-Pro4E-FS19T8-3DPrinterBoard-STM32-rescue:C-Device C103
 U 1 1 5CA6A17E
 P 4350 6900
@@
 	5700 6800 5700 7400
 $Comp
-L power:+24V #PWR?
+L FHNW-Pro4E-FS19T8-3DPrinterBoard-STM32-rescue:+24V-power #PWR?
 U 1 1 5CD67EF2
 P 2950 6300
@@
 $EndComp
 $Comp
-L Connector:Screw_Terminal_01x02 J101
+L FHNW-Pro4E-FS19T8-3DPrinterBoard-STM32-rescue:Screw_Terminal_01x02-Connector J101
 U 1 1 5CD68AD6
 P 650 6450
@@
 $EndBitmap
 $Comp
-L Regulator_Switching:LM2675M-3.3 U101
+L FHNW-Pro4E-FS19T8-3DPrinterBoard-STM32-rescue:LM2675M-3.3-Regulator_Switching U101
 U 1 1 5CA6A12A
 P 3650 6650
@@
 	2950 7250 3650 7250
 $Comp
-L Device:R R101
+L FHNW-Pro4E-FS19T8-3DPrinterBoard-STM32-rescue:R-Device R101
 U 1 1 5CB6A127
 P 6150 6700
@@
 $EndComp
 $Comp
-L Device:LED D102
+L FHNW-Pro4E-FS19T8-3DPrinterBoard-STM32-rescue:LED-Device D102
 U 1 1 5CB6AB63
 P 6150 7100
@@
 	5700 6450 6150 6450
 $Comp
-L power:GND #PWR0141
+L FHNW-Pro4E-FS19T8-3DPrinterBoard-STM32-rescue:GND-power #PWR0141
 U 1 1 5CB6C2A7
 P 6150 7400
@@
 	6150 7250 6150 7400
 $Comp
-L power:+3.3VP #PWR0121
+L FHNW-Pro4E-FS19T8-3DPrinterBoard-STM32-rescue:+3.3VP-power #PWR0121
 U 1 1 5CBF6320
 P 1800 3550
@@
 $EndComp
 $Comp
-L power:+3.3V #PWR0124
+L FHNW-Pro4E-FS19T8-3DPrinterBoard-STM32-rescue:+3.3V-power #PWR0124
 U 1 1 5CC01483
 P 1400 3600
@@
 $EndComp
 $Comp
-L power:+3.3VA #PWR0122
+L FHNW-Pro4E-FS19T8-3DPrinterBoard-STM32-rescue:+3.3VA-power #PWR0122
 U 1 1 5CC01489
 P 1000 3600
@@
 $EndComp
 $Comp
-L Device:Ferrite_Bead_Small FB?
+L FHNW-Pro4E-FS19T8-3DPrinterBoard-STM32-rescue:Ferrite_Bead_Small-Device FB?
 U 1 1 5CC0148F
 P 1000 3800
@@
 $EndComp
 $Comp
-L power:GND #PWR0125
+L FHNW-Pro4E-FS19T8-3DPrinterBoard-STM32-rescue:GND-power #PWR0125
 U 1 1 5CC014A8
 P 1000 4400
@@
 	1000 3950 1000 4000
 $Comp
-L Device:Ferrite_Bead_Small FB?
+L FHNW-Pro4E-FS19T8-3DPrinterBoard-STM32-rescue:Ferrite_Bead_Small-Device FB?
 U 1 1 5CC0728E
 P 1800 3800
@@
 	1800 3950 1400 3950
 $Comp
-L Device:C C106
+L FHNW-Pro4E-FS19T8-3DPrinterBoard-STM32-rescue:C-Device C106
 U 1 1 5CC0B14E
 P 1800 4150
@@
 $EndComp
 $Comp
-L power:GND #PWR0127
+L FHNW-Pro4E-FS19T8-3DPrinterBoard-STM32-rescue:GND-power #PWR0127
 U 1 1 5CC0B158
 P 1800 4400
@@
 	1400 3600 1400 3950
 $Comp
-L Device:C C104
+L FHNW-Pro4E-FS19T8-3DPrinterBoard-STM32-rescue:C-Device C104
 U 1 1 5CB61CA6
 P 1000 4150
@@
 	3800 5600 3650 5600
 $Comp
-L Device:D_Schottky D103
+L FHNW-Pro4E-FS19T8-3DPrinterBoard-STM32-rescue:D_Schottky-Device D103
 U 1 1 5CC3F964
 P 3950 5600
@@
 	3650 5400 3650 5600
 $Comp
-L power:GND #PWR0159
+L FHNW-Pro4E-FS19T8-3DPrinterBoard-STM32-rescue:GND-power #PWR0159
 U 1 1 5CC3F979
 P 5700 5750
@@
 $EndComp
 $Comp
-L power:GND #PWR0145
+L FHNW-Pro4E-FS19T8-3DPrinterBoard-STM32-rescue:GND-power #PWR0145
 U 1 1 5CC3F983
 P 2950 5750
@@
 $EndComp
 $Comp
-L Device:CP C107
+L FHNW-Pro4E-FS19T8-3DPrinterBoard-STM32-rescue:CP-Device C107
 U 1 1 5CC3F98D
 P 5700 5000
@@
 $EndComp
 $Comp
-L Device:L L102
+L FHNW-Pro4E-FS19T8-3DPrinterBoard-STM32-rescue:L-Device L102
 U 1 1 5CC3F997
 P 4900 5250
@@
 $EndComp
 $Comp
-L Device:CP C108
+L FHNW-Pro4E-FS19T8-3DPrinterBoard-STM32-rescue:CP-Device C108
 U 1 1 5CC3F9A1
 P 2950 5100
@@
 $EndComp
 $Comp
-L Device:C C109
+L FHNW-Pro4E-FS19T8-3DPrinterBoard-STM32-rescue:C-Device C109
 U 1 1 5CC3F9AB
 P 4350 5250
@@
 	5700 5150 5700 5750
 $Comp
-L power:+24V #PWR?
+L FHNW-Pro4E-FS19T8-3DPrinterBoard-STM32-rescue:+24V-power #PWR?
 U 1 1 5CC3F9D1
 P 2950 4650
@@
 	2950 5600 3650 5600
 $Comp
-L Regulator_Switching:LM2675M-5 U102
+L FHNW-Pro4E-FS19T8-3DPrinterBoard-STM32-rescue:LM2675M-5-Regulator_Switching U102
 U 1 1 5CC49DBB
 P 3650 5000
@@
 	3050 6450 2950 6450
 $Comp
-L power:+5V #PWR01
+L FHNW-Pro4E-FS19T8-3DPrinterBoard-STM32-rescue:+5V-power #PWR01
 U 1 1 5CBDFC0C
 P 5700 4650
@@
 $EndComp
 $Comp
-L Device:R R102
+L FHNW-Pro4E-FS19T8-3DPrinterBoard-STM32-rescue:R-Device R102
 U 1 1 5CC8B422
 P 6150 5050
@@
 $EndComp
 $Comp
-L Device:LED D104
+L FHNW-Pro4E-FS19T8-3DPrinterBoard-STM32-rescue:LED-Device D104
 U 1 1 5CC8B42C
 P 6150 5450
@@
 	5700 4800 6150 4800
 $Comp
-L power:GND #PWR0157
+L FHNW-Pro4E-FS19T8-3DPrinterBoard-STM32-rescue:GND-power #PWR0157
 U 1 1 5CC8B437
 P 6150 5750
@@
 	9700 4950 8650 4950
 $Comp
-L Mechanical:MountingHole H101
+L FHNW-Pro4E-FS19T8-3DPrinterBoard-STM32-rescue:MountingHole-Mechanical H101
 U 1 1 5CBF1F93
 P 850 750
@@
 $EndComp
 $Comp
-L Mechanical:MountingHole H102
+L FHNW-Pro4E-FS19T8-3DPrinterBoard-STM32-rescue:MountingHole-Mechanical H102
 U 1 1 5CBF3649
 P 1400 750
@@
 $EndComp
 $Comp
-L Mechanical:MountingHole H103
+L FHNW-Pro4E-FS19T8-3DPrinterBoard-STM32-rescue:MountingHole-Mechanical H103
 U 1 1 5CBF3A09
 P 850 1050
@@
 $EndComp
 $Comp
-L Mechanical:MountingHole H104
+L FHNW-Pro4E-FS19T8-3DPrinterBoard-STM32-rescue:MountingHole-Mechanical H104
 U 1 1 5CBF3E8E
 P 1400 1050
@@
 $EndComp
 $Comp
-L Device:R R103
+L FHNW-Pro4E-FS19T8-3DPrinterBoard-STM32-rescue:R-Device R103
 U 1 1 5CCAE006
 P 1900 6700
@@
 	1900 6450 1900 6550
 $Comp
-L Device:D_Zener D105
+L FHNW-Pro4E-FS19T8-3DPrinterBoard-STM32-rescue:D_Zener-Device D105
 U 1 1 5CD1A22D
 P 2250 7100
@@
 	2250 6950 2250 6900
 $Comp
-L Device:Fuse F?
+L FHNW-Pro4E-FS19T8-3DPrinterBoard-STM32-rescue:Fuse-Device F?
 U 1 1 5CE8417C
 P 2500 6450
@@
 24V_IN
 $Comp
-L Device:R R104
+L FHNW-Pro4E-FS19T8-3DPrinterBoard-STM32-rescue:R-Device R104
 U 1 1 5CC041F6
 P 1450 6300
@@
 $EndComp
 $Comp
-L SparkFun-Aesthetics:OSHW-LOGOM-COPPER LOGO101
+L FHNW-Pro4E-FS19T8-3DPrinterBoard-STM32-rescue:OSHW-LOGOM-COPPER-SparkFun-Aesthetics LOGO101
 U 1 1 5CC5A1CC
 P 1200 2300
@@
 	4500 2550 4200 2550
 $Comp
-L power:PWR_FLAG #FLG0101
+L FHNW-Pro4E-FS19T8-3DPrinterBoard-STM32-rescue:PWR_FLAG-power #FLG0101
 U 1 1 5E688628
 P 700 5000
@@
 $EndComp
 $Comp
-L power:+3.3VA #PWR0126
+L FHNW-Pro4E-FS19T8-3DPrinterBoard-STM32-rescue:+3.3VA-power #PWR0126
 U 1 1 5E68AEEF
 P 700 5000
@@
 $EndComp
 $Comp
-L power:PWR_FLAG #FLG0102
+L FHNW-Pro4E-FS19T8-3DPrinterBoard-STM32-rescue:PWR_FLAG-power #FLG0102
 U 1 1 5E693379
 P 1000 5000
@@
 $EndComp
 $Comp
-L power:+3.3V #PWR0237
+L FHNW-Pro4E-FS19T8-3DPrinterBoard-STM32-rescue:+3.3V-power #PWR0237
 U 1 1 5E69357A
 P 1000 5000
@@
 $EndComp
 $Comp
-L power:+3.3VP #PWR0246
+L FHNW-Pro4E-FS19T8-3DPrinterBoard-STM32-rescue:+3.3VP-power #PWR0246
 U 1 1 5E69A805
 P 1300 5000
@@
 $EndComp
 $Comp
-L power:PWR_FLAG #FLG0103
+L FHNW-Pro4E-FS19T8-3DPrinterBoard-STM32-rescue:PWR_FLAG-power #FLG0103
 U 1 1 5E69AB83
 P 1300 5000
@@
 $EndComp
 $Comp
-L power:+24V #PWR?
+L FHNW-Pro4E-FS19T8-3DPrinterBoard-STM32-rescue:+24V-power #PWR?
 U 1 1 5E69ACDE
 P 1600 5000
@@
 $EndComp
 $Comp
-L power:PWR_FLAG #FLG0104
+L FHNW-Pro4E-FS19T8-3DPrinterBoard-STM32-rescue:PWR_FLAG-power #FLG0104
 U 1 1 5E69B096
 P 1600 5000
@@
 $EndComp
 $Comp
-L power:PWR_FLAG #FLG0105
+L FHNW-Pro4E-FS19T8-3DPrinterBoard-STM32-rescue:PWR_FLAG-power #FLG0105
 U 1 1 5E6A206A
 P 1900 5000
@@
 $EndComp
 $Comp
-L power:+5V #PWR0265
+L FHNW-Pro4E-FS19T8-3DPrinterBoard-STM32-rescue:+5V-power #PWR0265
 U 1 1 5E6A2352
 P 1900 5000
@@
 $EndComp
 $Comp
-L power:VBUS #PWR?
+L FHNW-Pro4E-FS19T8-3DPrinterBoard-STM32-rescue:VBUS-power #PWR?
 U 1 1 5E6AB26A
 P 2200 5000
@@
 $EndComp
 $Comp
-L power:PWR_FLAG #FLG0106
+L FHNW-Pro4E-FS19T8-3DPrinterBoard-STM32-rescue:PWR_FLAG-power #FLG0106
 U 1 1 5E6BE425
 P 2200 5000
@@
 	-1   0    0    1
 $EndComp
+Text Notes 6300 5650 0    50   ~ 10
+GREEN
+Text Notes 900  3300 0    50   ~ 10
+C104 misplaced on the PCB,\nshould be near +3.3VA
+Text Notes 2400 6600 0    50   ~ 10
+20A
+Text Notes 6300 7300 0    50   ~ 10
+GREEN
 $EndSCHEMATC
