File: appendix_UART_USB.sch (KiCad schematic (older format))
At the start: 0 parts

Commit message: added FTDI chip
Parts:
- added J?: USB_B_Mini, symbol Connector:USB_B_Mini
- added J? (x2): Conn_01x04, symbol Connector_Generic:Conn_01x04
- added L?: Ferrite_Bead, symbol Device:Ferrite_Bead_Small
- added R? (x2): 10k, symbol Device:R
- added R?: 4k7, symbol Device:R
- added U?: FT232RL, Package_SO:SSOP-28_5.3x10.2mm_P0.65mm, symbol FHNW-Pro4E-FS19T8-Library:FT232RL
Connections:
- net labels added: +3V3, +5V, D_RX_to_USB_TX, D_TX_to_USB_RX, USB_DM, USB_DP, USB_VBUS
- net labels removed: +3.3V
- wire segments 0 -> 34
- no-connect marks 0 -> 13

Commit message: pre Annotation 1
Connections:
- net labels added: DTR_ESP32, D_FTDI_DTR, D_FTDI_RTS, RTS_ESP32
- wire segments 34 -> 38
- no-connect marks 13 -> 11
Changed lines of the file:
@@
 $Descr A4 11693 8268
 encoding utf-8
-Sheet 6 7
+Sheet 5 6
 Title "USB to UART Interface"
 Date ""
@@
 Text GLabel 9250 4200 0    50   Input ~ 0
 D_TX_to_USB_RX
-NoConn ~ 6650 3650
-NoConn ~ 6650 3750
-NoConn ~ 6650 3850
 NoConn ~ 6650 3950
 NoConn ~ 6650 4050
@@
 EndData
 $EndBitmap
+Text HLabel 7950 2200 0    50   Input ~ 0
+DTR_ESP32
+Text HLabel 7950 2100 0    50   Input ~ 0
+RTS_ESP32
+Text GLabel 6800 3650 2    50   Input ~ 0
+D_FTDI_RTS
+Text GLabel 6800 3850 2    50   Input ~ 0
+D_FTDI_DTR
+Wire Wire Line
+	6650 3850 6800 3850
+Text GLabel 8100 2100 2    50   Input ~ 0
+D_FTDI_RTS
+Text GLabel 8100 2200 2    50   Input ~ 0
+D_FTDI_DTR
+Wire Wire Line
+	6650 3650 6800 3650
+NoConn ~ 6650 3750
+Wire Wire Line
+	7950 2100 8100 2100
+Wire Wire Line
+	7950 2200 8100 2200
 $EndSCHEMATC

Commit message: 1st annotation, footprints, netlist
Parts:
- J501: renamed from J?; footprint (none) -> Connector_PinHeader_2.54mm:PinHeader_1x04_P2.54mm_Vertical_SMD_Pin1Left
- J502: renamed from J?; footprint (none) -> Connector_USB:USB_Mini-B_Lumberg_2486_01_Horizontal
- J503: renamed from J?; footprint (none) -> Connector_PinHeader_2.54mm:PinHeader_1x04_P2.54mm_Vertical
- L501: renamed from L?; footprint (none) -> Resistors_SMD:R_0805_HandSoldering
- R501, R502, R503: renamed from R?; footprint (none) -> Resistors_SMD:R_0805
- U501: renamed from U?; footprint Package_SO:SSOP-28_5.3x10.2mm_P0.65mm -> Housings_SSOP:SSOP-28_5.3x10.2mm_Pitch0.65mm
Changed lines of the file:
@@
 $EndDescr
 $Comp
-L power:GND #PWR?
+L power:GND #PWR0157
 U 1 1 5CA3CCA1
 P 5850 5350
-F 0 "#PWR?" H 5850 5100 50  0001 C CNN
+F 0 "#PWR0157" H 5850 5100 50  0001 C CNN
 F 1 "GND" H 5855 5177 50  0000 C CNN
 F 2 "" H 5850 5350 50  0001 C CNN
@@
 D_RX_to_STM_TX
 $Comp
-L FHNW-Pro4E-FS19T8-Library:FT232RL U?
+L FHNW-Pro4E-FS19T8-Library:FT232RL U501
 U 1 1 5CA46716
 P 5850 4150
-F 0 "U?" H 6300 5100 50  0000 C CNN
+F 0 "U501" H 6300 5100 50  0000 C CNN
 F 1 "FT232RL" H 5850 4050 50  0000 C CNN
-F 2 "Package_SO:SSOP-28_5.3x10.2mm_P0.65mm" H 5850 4150 50  0001 C CNN
+F 2 "Housings_SSOP:SSOP-28_5.3x10.2mm_Pitch0.65mm" H 5850 4150 50  0001 C CNN
 F 3 "" H 5850 4150 50  0001 C CNN
 	1    5850 4150
@@
 NoConn ~ 5050 4350
 $Comp
-L Device:R R?
+L Device:R R502
 U 1 1 5CA469B4
 P 7050 4550
-F 0 "R?" H 7120 4596 50  0000 L CNN
+F 0 "R502" H 7120 4596 50  0000 L CNN
 F 1 "10k" H 7120 4505 50  0000 L CNN
-F 2 "" V 6980 4550 50  0001 C CNN
+F 2 "Resistors_SMD:R_0805" V 6980 4550 50  0001 C CNN
 F 3 "~" H 7050 4550 50  0001 C CNN
 	1    7050 4550
@@
 $EndComp
 $Comp
-L Device:R R?
+L Device:R R503
 U 1 1 5CA46A3C
 P 4500 4600
-F 0 "R?" H 4570 4646 50  0000 L CNN
+F 0 "R503" H 4570 4646 50  0000 L CNN
 F 1 "10k" H 4570 4555 50  0000 L CNN
-F 2 "" V 4430 4600 50  0001 C CNN
+F 2 "Resistors_SMD:R_0805" V 4430 4600 50  0001 C CNN
 F 3 "~" H 4500 4600 50  0001 C CNN
 	1    4500 4600
@@
 $EndComp
 $Comp
-L Device:R R?
+L Device:R R501
 U 1 1 5CA46A68
 P 4500 4200
-F 0 "R?" H 4570 4246 50  0000 L CNN
+F 0 "R501" H 4570 4246 50  0000 L CNN
 F 1 "4k7" H 4570 4155 50  0000 L CNN
-F 2 "" V 4430 4200 50  0001 C CNN
+F 2 "Resistors_SMD:R_0805" V 4430 4200 50  0001 C CNN
 F 3 "~" H 4500 4200 50  0001 C CNN
 	1    4500 4200
@@
 	4500 4400 4500 4350
 $Comp
-L power:GND #PWR?
+L power:GND #PWR0158
 U 1 1 5CA46C75
 P 4500 4850
-F 0 "#PWR?" H 4500 4600 50  0001 C CNN
+F 0 "#PWR0158" H 4500 4600 50  0001 C CNN
 F 1 "GND" H 4505 4677 50  0000 C CNN
 F 2 "" H 4500 4850 50  0001 C CNN
@@
 	4500 4850 4500 4750
 $Comp
-L Connector:USB_B_Mini J?
+L Connector:USB_B_Mini J502
 U 1 1 5CA4790B
 P 3650 3750
-F 0 "J?" H 3705 4217 50  0000 C CNN
+F 0 "J502" H 3705 4217 50  0000 C CNN
 F 1 "USB_B_Mini" H 3705 4126 50  0000 C CNN
-F 2 "" H 3800 3700 50  0001 C CNN
+F 2 "Connector_USB:USB_Mini-B_Lumberg_2486_01_Horizontal" H 3800 3700 50  0001 C CNN
 F 3 "~" H 3800 3700 50  0001 C CNN
 	1    3650 3750
@@
 	4500 3550 3950 3550
 $Comp
-L power:GND #PWR?
+L power:GND #PWR0159
 U 1 1 5CA480FD
 P 3650 4850
-F 0 "#PWR?" H 3650 4600 50  0001 C CNN
+F 0 "#PWR0159" H 3650 4600 50  0001 C CNN
 F 1 "GND" H 3655 4677 50  0000 C CNN
 F 2 "" H 3650 4850 50  0001 C CNN
@@
 Connection ~ 3650 4650
 $Comp
-L Device:Ferrite_Bead_Small L?
+L Device:Ferrite_Bead_Small L501
 U 1 1 5CA48BE5
 P 3550 4400
-F 0 "L?" H 3300 4450 50  0000 L CNN
+F 0 "L501" H 3300 4450 50  0000 L CNN
 F 1 "Ferrite_Bead" H 2950 4350 50  0000 L CNN
-F 2 "" V 3480 4400 50  0001 C CNN
+F 2 "Resistors_SMD:R_0805_HandSoldering" V 3480 4400 50  0001 C CNN
 F 3 "~" H 3550 4400 50  0001 C CNN
 	1    3550 4400
@@
 NoConn ~ 3950 3950
 $Comp
-L power:+3V3 #PWR?
+L power:+3V3 #PWR0160
 U 1 1 5CA49DB7
 P 5750 3050
-F 0 "#PWR?" H 5750 2900 50  0001 C CNN
+F 0 "#PWR0160" H 5750 2900 50  0001 C CNN
 F 1 "+3V3" H 5765 3223 50  0000 C CNN
 F 2 "" H 5750 3050 50  0001 C CNN
@@
 USB_VBUS
 $Comp
-L power:+3V3 #PWR?
+L power:+3V3 #PWR0161
 U 1 1 5CA4A848
 P 7050 4300
-F 0 "#PWR?" H 7050 4150 50  0001 C CNN
+F 0 "#PWR0161" H 7050 4150 50  0001 C CNN
 F 1 "+3V3" H 7065 4473 50  0000 C CNN
 F 2 "" H 7050 4300 50  0001 C CNN
@@
 NoConn ~ 6650 4450
 $Comp
-L Connector_Generic:Conn_01x04 J?
+L Connector_Generic:Conn_01x04 J501
 U 1 1 5CA4CA0C
 P 9450 3500
-F 0 "J?" H 9530 3492 50  0000 L CNN
+F 0 "J501" H 9530 3492 50  0000 L CNN
 F 1 "Conn_01x04" H 9530 3401 50  0000 L CNN
-F 2 "" H 9450 3500 50  0001 C CNN
+F 2 "Connector_PinHeader_2.54mm:PinHeader_1x04_P2.54mm_Vertical_SMD_Pin1Left" H 9450 3500 50  0001 C CNN
 F 3 "~" H 9450 3500 50  0001 C CNN
 	1    9450 3500
@@
 $EndComp
 $Comp
-L Connector_Generic:Conn_01x04 J?
+L Connector_Generic:Conn_01x04 J503
 U 1 1 5CA4CFF7
 P 9450 4100
-F 0 "J?" H 9530 4092 50  0000 L CNN
+F 0 "J503" H 9530 4092 50  0000 L CNN
 F 1 "Conn_01x04" H 9530 4001 50  0000 L CNN
-F 2 "" H 9450 4100 50  0001 C CNN
+F 2 "Connector_PinHeader_2.54mm:PinHeader_1x04_P2.54mm_Vertical" H 9450 4100 50  0001 C CNN
 F 3 "~" H 9450 4100 50  0001 C CNN
 	1    9450 4100
@@
 NoConn ~ 6650 4150
 $Comp
-L power:+5V #PWR?
+L power:+5V #PWR0162
 U 1 1 5CA4FF52
 P 5950 3050
-F 0 "#PWR?" H 5950 2900 50  0001 C CNN
+F 0 "#PWR0162" H 5950 2900 50  0001 C CNN
 F 1 "+5V" H 5965 3223 50  0000 C CNN
 F 2 "" H 5950 3050 50  0001 C CNN
@@
 	5950 3050 5950 3150
 $Comp
-L power:+5V #PWR?
+L power:+5V #PWR0163
 U 1 1 5CA50457
 P 4500 3350
-F 0 "#PWR?" H 4500 3200 50  0001 C CNN
+F 0 "#PWR0163" H 4500 3200 50  0001 C CNN
 F 1 "+5V" H 4515 3523 50  0000 C CNN
 F 2 "" H 4500 3350 50  0001 C CNN

Commit message: started layouting TMC2660
Parts:
- added C501: 10n, Capacitors_SMD:C_0603, symbol Device:C
- added C502, C504: 100n, Capacitors_SMD:C_0603, symbol Device:C
- added C503: 4.7u, Capacitor_SMD:CP_Elec_6.3x5.3, symbol Device:CP
- added L502: Ferrite_Bead, Resistors_SMD:R_0805_HandSoldering, symbol Device:Ferrite_Bead_Small
- R501, R502, R503: footprint Resistors_SMD:R_0805 -> Resistors_SMD:R_0603
Connections:
- net labels added: USB_VCCIO_3.3V, V_USB
- net labels removed: +3V3, +5V, USB_VBUS
- wire segments 38 -> 48
Other:
- moved on the sheet: L501

Commit message: added footprints, layouted 3v3 Reg
Parts:
- C503: footprint Capacitor_SMD:CP_Elec_6.3x5.3 -> Capacitor_SMD:CP_Elec_5x5.9
- J501: footprint Connector_PinHeader_2.54mm:PinHeader_1x04_P2.54mm_Vertical_SMD_Pin1Left -> Connector_PinHeader_2.54mm:PinHeader_1x04_P2.54mm_Vertical
Connections:
- net labels added: USB_D_N, USB_D_P
- net labels removed: USB_DM, USB_DP

Commit message: corrected P.S. Schematic review
Parts:
- removed C501: 10n, Capacitors_SMD:C_0603, symbol Device:C
- removed J502: USB_B_Mini, Connector_USB:USB_Mini-B_Lumberg_2486_01_Horizontal, symbol Connector:USB_B_Mini
- removed L501: Ferrite_Bead, Resistors_SMD:R_0805_HandSoldering, symbol Device:Ferrite_Bead_Small
- added D501: USBLC6-2SC6, digikey-footprints:SOT23-6L, symbol dk_TVS-Diodes:USBLC6-2SC6
- added F501: MF-MSMF050-2, symbol Device:Polyfuse
- added FB501: Ferrite_Bead, symbol Device:Ferrite_Bead
- added J504: USB_C_Receptacle, Connector_USB:USB_C_Receptacle_GCT_USB4085, symbol Connector:USB_C_Receptacle
- added L501: WE-744232090, symbol FHNW-Pro4E-FS19T8-Library:WE-744232090
- added R504, R505: 22R, Resistors_SMD:R_0603, symbol Device:R
Connections:
- net labels added: 5V, USB_D_SUP_N, USB_D_SUP_P, USB_D_TVS_N, USB_D_TVS_P, VBUS
- wire segments 48 -> 66
- no-connect marks 11 -> 10
Other:
- note added: "Jumper to select \nUART communication"
- moved on the sheet: C502, J501, J503, L502, R501, R502, R503

Commit message: added FT2232 by Marco M
Parts:
- removed C503: 4.7u, Capacitor_SMD:CP_Elec_5x5.9, symbol Device:CP
- removed F501: MF-MSMF050-2, symbol Device:Polyfuse
- removed FB501: Ferrite_Bead, symbol Device:Ferrite_Bead
- removed J501, J503: Conn_01x04, Connector_PinHeader_2.54mm:PinHeader_1x04_P2.54mm_Vertical, symbol Connector_Generic:Conn_01x04
- removed L502: Ferrite_Bead, Resistors_SMD:R_0805_HandSoldering, symbol Device:Ferrite_Bead_Small
- removed U501: FT232RL, Housings_SSOP:SSOP-28_5.3x10.2mm_Pitch0.65mm, symbol FHNW-Pro4E-FS19T8-Library:FT232RL
- added C501, C505, C506: 100n, Capacitors_SMD:C_0603, symbol Device:C
- added C503: 10n, Capacitors_SMD:C_0603, symbol Device:C
- added C507: 10u, Capacitors_SMD:C_1210, symbol Device:CP
- added D502, D503, D504, D505: LED, LED_SMD:LED_0805_2012Metric, symbol Device:LED
- added R506, R507: 10k, Resistors_SMD:R_0603, symbol Device:R
- added R508, R509, R510, R511: 330R, Resistors_SMD:R_0603, symbol Device:R
- added U502: FT2232D, Package_QFP:LQFP-48_7x7mm_P0.5mm, symbol Interface_USB:FT2232D
- added X501: SG5032CCN-6.000000M-HJGA3, Oscillator:Oscillator_SMD_SeikoEpson_SG8002LB-4Pin_5.0x3.2mm, symbol FHNW-Pro4E-FS19T8-Library:SG5032CCN-6.000000M-HJGA3
- R501: value 4k7 -> 470R
- R502: value 10k -> 1k5
- R503: value 10k -> 4k7
- R504, R505: value 22R -> 27R
Connections:
- net labels added: 3.3V, RX_ESP_to_TX_FTDI, RX_STM_to_TX_FTDI, TX_ESP_to_RX_FTDI, TX_STM_to_RX_FTDI, UART1_RX_LED, UART1_TX_LED, UART2_RX_LED, UART2_TX_LED, USB_FT_D_N, USB_FT_D_P, USB_SUP_D_N, USB_SUP_D_P, USB_TVS_D_N, USB_TVS_D_P, XTAL_FTDI
- net labels removed: D_FTDI_DTR, D_FTDI_RTS, D_RX_to_ESP_TX, D_RX_to_STM_TX, D_RX_to_USB_TX, D_TX_to_ESP_RX, D_TX_to_STM_RX, D_TX_to_USB_RX, USB_D_SUP_N, USB_D_SUP_P, USB_D_TVS_N, USB_D_TVS_P, USB_VCCIO_3.3V, V_USB
- wire segments 66 -> 111
- no-connect marks 10 -> 18
Other:
- note removed: "Jumper to select \nUART communication"
- moved on the sheet: C502, J504, L501, R504, R505
