File: appendix_UART_USB.sch (KiCad schematic (older format))
At the start: 29 parts, among them J504 USB_C_Receptacle, U1 USBLC6-2SC6, U502 FT2232D, X501 SG5032CCN-6.000000M-HJGA3

Commit message: Added comments to the schematic. Changed various component values (annotated only).
Parts:
- C1, C501, C502, C503, C504, C505, C506, C508: symbol Device:C -> FHNW-Pro4E-FS19T8-3DPrinterBoard-STM32-rescue:C-Device
- C507: symbol Device:CP -> FHNW-Pro4E-FS19T8-3DPrinterBoard-STM32-rescue:CP-Device
- D502, D503, D504, D505: symbol Device:LED -> FHNW-Pro4E-FS19T8-3DPrinterBoard-STM32-rescue:LED-Device
- J504: symbol Connector:USB_C_Receptacle -> FHNW-Pro4E-FS19T8-3DPrinterBoard-STM32-rescue:USB_C_Receptacle-Connector
- R501, R502, R503, R504, R505, R506, R507, R508, R509, R510, R511: symbol Device:R -> FHNW-Pro4E-FS19T8-3DPrinterBoard-STM32-rescue:R-Device
- U1: symbol Power_Protection:USBLC6-2SC6 -> FHNW-Pro4E-FS19T8-3DPrinterBoard-STM32-rescue:USBLC6-2SC6-Power_Protection
- U502: symbol Interface_USB:FT2232D -> FHNW-Pro4E-FS19T8-3DPrinterBoard-STM32-rescue:FT2232D-Interface_USB
Other:
- note added: "100n"
- note added: "YELLOW"
Changed lines of the file:
@@
 $EndDescr
 $Comp
-L Device:C C502
+L FHNW-Pro4E-FS19T8-3DPrinterBoard-STM32-rescue:C-Device C502
 U 1 1 5CCC5851
 P 1450 6950
@@
 $EndBitmap
 $Comp
-L Connector:USB_C_Receptacle J504
+L FHNW-Pro4E-FS19T8-3DPrinterBoard-STM32-rescue:USB_C_Receptacle-Connector J504
 U 1 1 5CB2E973
 P 1100 2700
@@
 $EndComp
 $Comp
-L power:GND #PWR0143
+L FHNW-Pro4E-FS19T8-3DPrinterBoard-STM32-rescue:GND-power #PWR0143
 U 1 1 5CB335A4
 P 1100 4400
@@
 	1750 2200 1700 2200
 $Comp
-L power:GND #PWR0508
+L FHNW-Pro4E-FS19T8-3DPrinterBoard-STM32-rescue:GND-power #PWR0508
 U 1 1 5CB6D401
 P 800 4400
@@
 	800  4400 800  4300
 $Comp
-L power:VBUS #PWR0501
+L FHNW-Pro4E-FS19T8-3DPrinterBoard-STM32-rescue:VBUS-power #PWR0501
 U 1 1 5CB8117C
 P 1800 1600
@@
 USB_D_N
 $Comp
-L power:GND #PWR0507
+L FHNW-Pro4E-FS19T8-3DPrinterBoard-STM32-rescue:GND-power #PWR0507
 U 1 1 5CB8B8DF
 P 1450 7200
@@
 $EndComp
 $Comp
-L power:VBUS #PWR0506
+L FHNW-Pro4E-FS19T8-3DPrinterBoard-STM32-rescue:VBUS-power #PWR0506
 U 1 1 5CB8BCC6
 P 1450 6700
@@
 $EndComp
 $Comp
-L Device:R R504
+L FHNW-Pro4E-FS19T8-3DPrinterBoard-STM32-rescue:R-Device R504
 U 1 1 5CB9736D
 P 5450 2250
@@
 $EndComp
 $Comp
-L Device:R R505
+L FHNW-Pro4E-FS19T8-3DPrinterBoard-STM32-rescue:R-Device R505
 U 1 1 5CB99459
 P 5450 2450
@@
 USB_SUP_D_N
 $Comp
-L Interface_USB:FT2232D U502
+L FHNW-Pro4E-FS19T8-3DPrinterBoard-STM32-rescue:FT2232D-Interface_USB U502
 U 1 1 5CB6FC61
 P 7100 3150
@@
 USB_FT_D_N
 $Comp
-L power:GND #PWR0509
+L FHNW-Pro4E-FS19T8-3DPrinterBoard-STM32-rescue:GND-power #PWR0509
 U 1 1 5CBA3BBE
 P 7100 5050
@@
 NoConn ~ 8000 3450
 $Comp
-L Device:R R501
+L FHNW-Pro4E-FS19T8-3DPrinterBoard-STM32-rescue:R-Device R501
 U 1 1 5CBEADDA
 P 6700 1050
@@
 Connection ~ 7200 1200
 $Comp
-L Device:C C501
+L FHNW-Pro4E-FS19T8-3DPrinterBoard-STM32-rescue:C-Device C501
 U 1 1 5CBFAF1C
 P 6250 1250
@@
 $EndComp
 $Comp
-L power:GND #PWR0502
+L FHNW-Pro4E-FS19T8-3DPrinterBoard-STM32-rescue:GND-power #PWR0502
 U 1 1 5CBFC058
 P 6050 1300
@@
 	4600 2450 5300 2450
 $Comp
-L Device:R R502
+L FHNW-Pro4E-FS19T8-3DPrinterBoard-STM32-rescue:R-Device R502
 U 1 1 5CC34C99
 P 6050 2650
@@
 	6050 2850 6200 2850
 $Comp
-L power:VBUS #PWR0503
+L FHNW-Pro4E-FS19T8-3DPrinterBoard-STM32-rescue:VBUS-power #PWR0503
 U 1 1 5CC418C4
 P 5000 2750
@@
 $EndComp
 $Comp
-L Device:R R503
+L FHNW-Pro4E-FS19T8-3DPrinterBoard-STM32-rescue:R-Device R503
 U 1 1 5CC422DE
 P 5000 2900
@@
 $EndComp
 $Comp
-L Device:R R506
+L FHNW-Pro4E-FS19T8-3DPrinterBoard-STM32-rescue:R-Device R506
 U 1 1 5CC4295B
 P 5000 3200
@@
 Connection ~ 5000 3050
 $Comp
-L power:GND #PWR0510
+L FHNW-Pro4E-FS19T8-3DPrinterBoard-STM32-rescue:GND-power #PWR0510
 U 1 1 5CC47BA9
 P 5000 3350
@@
 $EndComp
 $Comp
-L Device:R R507
+L FHNW-Pro4E-FS19T8-3DPrinterBoard-STM32-rescue:R-Device R507
 U 1 1 5CC49179
 P 5950 4250
@@
 	5750 4250 5800 4250
 $Comp
-L Device:LED D?
+L FHNW-Pro4E-FS19T8-3DPrinterBoard-STM32-rescue:LED-Device D?
 U 1 1 5CC68B5F
 P 9350 4850
@@
 $EndComp
 $Comp
-L Device:R R508
+L FHNW-Pro4E-FS19T8-3DPrinterBoard-STM32-rescue:R-Device R508
 U 1 1 5CC6C674
 P 9350 5200
@@
 	9350 5350 9350 5450
 $Comp
-L Device:LED D?
+L FHNW-Pro4E-FS19T8-3DPrinterBoard-STM32-rescue:LED-Device D?
 U 1 1 5CC8BE19
 P 9800 4850
@@
 $EndComp
 $Comp
-L Device:R R509
+L FHNW-Pro4E-FS19T8-3DPrinterBoard-STM32-rescue:R-Device R509
 U 1 1 5CC8BE2D
 P 9800 5200
@@
 	9800 5350 9800 5450
 $Comp
-L Device:LED D?
+L FHNW-Pro4E-FS19T8-3DPrinterBoard-STM32-rescue:LED-Device D?
 U 1 1 5CC90F6E
 P 10250 4850
@@
 $EndComp
 $Comp
-L Device:R R510
+L FHNW-Pro4E-FS19T8-3DPrinterBoard-STM32-rescue:R-Device R510
 U 1 1 5CC90F82
 P 10250 5200
@@
 	10250 5350 10250 5450
 $Comp
-L Device:LED D?
+L FHNW-Pro4E-FS19T8-3DPrinterBoard-STM32-rescue:LED-Device D?
 U 1 1 5CC90F8F
 P 10700 4850
@@
 $EndComp
 $Comp
-L Device:R R511
+L FHNW-Pro4E-FS19T8-3DPrinterBoard-STM32-rescue:R-Device R511
 U 1 1 5CC90FA3
 P 10700 5200
@@
 $EndComp
 $Comp
-L Device:C C503
+L FHNW-Pro4E-FS19T8-3DPrinterBoard-STM32-rescue:C-Device C503
 U 1 1 5CC9F50E
 P 3950 4200
@@
 $EndComp
 $Comp
-L power:+5V #SUPPLY0502
+L FHNW-Pro4E-FS19T8-3DPrinterBoard-STM32-rescue:+5V-power #SUPPLY0502
 U 1 1 5CCA003E
 P 4100 3800
@@
 	4500 4550 4500 4500
 $Comp
-L power:GND #PWR0511
+L FHNW-Pro4E-FS19T8-3DPrinterBoard-STM32-rescue:GND-power #PWR0511
 U 1 1 5CCBF21B
 P 4500 4600
@@
 	1450 7200 1450 7100
 $Comp
-L Device:C C504
+L FHNW-Pro4E-FS19T8-3DPrinterBoard-STM32-rescue:C-Device C504
 U 1 1 5CD73761
 P 1950 6950
@@
 $EndComp
 $Comp
-L power:GND #PWR0512
+L FHNW-Pro4E-FS19T8-3DPrinterBoard-STM32-rescue:GND-power #PWR0512
 U 1 1 5CD7376B
 P 1950 7200
@@
 	1950 7200 1950 7100
 $Comp
-L Device:C C505
+L FHNW-Pro4E-FS19T8-3DPrinterBoard-STM32-rescue:C-Device C505
 U 1 1 5CD79248
 P 2750 6950
@@
 $EndComp
 $Comp
-L power:GND #PWR0513
+L FHNW-Pro4E-FS19T8-3DPrinterBoard-STM32-rescue:GND-power #PWR0513
 U 1 1 5CD79252
 P 2750 7200
@@
 	2750 7200 2750 7100
 $Comp
-L Device:C C506
+L FHNW-Pro4E-FS19T8-3DPrinterBoard-STM32-rescue:C-Device C506
 U 1 1 5CD7CE0B
 P 3200 6950
@@
 $EndComp
 $Comp
-L power:GND #PWR0514
+L FHNW-Pro4E-FS19T8-3DPrinterBoard-STM32-rescue:GND-power #PWR0514
 U 1 1 5CD7CE15
 P 3200 7200
@@
 	3200 7200 3200 7100
 $Comp
-L power:GND #PWR0515
+L FHNW-Pro4E-FS19T8-3DPrinterBoard-STM32-rescue:GND-power #PWR0515
 U 1 1 5CD80C48
 P 3650 7200
@@
 	3650 7200 3650 7100
 $Comp
-L Device:CP C507
+L FHNW-Pro4E-FS19T8-3DPrinterBoard-STM32-rescue:CP-Device C507
 U 1 1 5CD84D48
 P 3650 6950
@@
 $EndBitmap
 $Comp
-L power:+3.3V #PWR05
+L FHNW-Pro4E-FS19T8-3DPrinterBoard-STM32-rescue:+3.3V-power #PWR05
 U 1 1 5CBC6C94
 P 1950 6700
@@
 $EndComp
 $Comp
-L power:+5V #PWR06
+L FHNW-Pro4E-FS19T8-3DPrinterBoard-STM32-rescue:+5V-power #PWR06
 U 1 1 5CBC8577
 P 2750 6700
@@
 $EndComp
 $Comp
-L power:+5V #PWR07
+L FHNW-Pro4E-FS19T8-3DPrinterBoard-STM32-rescue:+5V-power #PWR07
 U 1 1 5CBC9FB7
 P 3200 6700
@@
 $EndComp
 $Comp
-L power:+5V #PWR08
+L FHNW-Pro4E-FS19T8-3DPrinterBoard-STM32-rescue:+5V-power #PWR08
 U 1 1 5CBCA403
 P 3650 6700
@@
 $EndComp
 $Comp
-L power:+3.3V #PWR014
+L FHNW-Pro4E-FS19T8-3DPrinterBoard-STM32-rescue:+3.3V-power #PWR014
 U 1 1 5CBCCA6E
 P 9350 4650
@@
 $EndComp
 $Comp
-L power:+3.3V #PWR015
+L FHNW-Pro4E-FS19T8-3DPrinterBoard-STM32-rescue:+3.3V-power #PWR015
 U 1 1 5CBCDEA6
 P 9800 4650
@@
 $EndComp
 $Comp
-L power:+3.3V #PWR016
+L FHNW-Pro4E-FS19T8-3DPrinterBoard-STM32-rescue:+3.3V-power #PWR016
 U 1 1 5CBCE321
 P 10250 4650
@@
 $EndComp
 $Comp
-L power:+3.3V #PWR017
+L FHNW-Pro4E-FS19T8-3DPrinterBoard-STM32-rescue:+3.3V-power #PWR017
 U 1 1 5CBCE6EF
 P 10700 4650
@@
 $EndComp
 $Comp
-L power:+3.3V #PWR013
+L FHNW-Pro4E-FS19T8-3DPrinterBoard-STM32-rescue:+3.3V-power #PWR013
 U 1 1 5CBCEAA3
 P 8150 4450
@@
 $EndComp
 $Comp
-L power:+3.3V #PWR012
+L FHNW-Pro4E-FS19T8-3DPrinterBoard-STM32-rescue:+3.3V-power #PWR012
 U 1 1 5CBD2E53
 P 8150 2950
@@
 $EndComp
 $Comp
-L power:+3.3V #PWR011
+L FHNW-Pro4E-FS19T8-3DPrinterBoard-STM32-rescue:+3.3V-power #PWR011
 U 1 1 5CBD3B4C
 P 7200 800
@@
 $EndComp
 $Comp
-L power:+5V #PWR09
+L FHNW-Pro4E-FS19T8-3DPrinterBoard-STM32-rescue:+5V-power #PWR09
 U 1 1 5CBD4A5B
 P 5750 4250
@@
 $EndComp
 $Comp
-L power:+5V #PWR010
+L FHNW-Pro4E-FS19T8-3DPrinterBoard-STM32-rescue:+5V-power #PWR010
 U 1 1 5CBD5B3B
 P 6900 800
@@
 $EndComp
 $Comp
-L Device:C C1
+L FHNW-Pro4E-FS19T8-3DPrinterBoard-STM32-rescue:C-Device C1
 U 1 1 5CBC7319
 P 6050 1850
@@
 	6050 1250 6100 1250
 $Comp
-L power:GND #PWR018
+L FHNW-Pro4E-FS19T8-3DPrinterBoard-STM32-rescue:GND-power #PWR018
 U 1 1 5CBD5EB7
 P 5850 1900
@@
 FT_RTS_B
 $Comp
-L power:GND #PWR0504
+L FHNW-Pro4E-FS19T8-3DPrinterBoard-STM32-rescue:GND-power #PWR0504
 U 1 1 5CC897FA
 P 2450 2350
@@
 $EndComp
 $Comp
-L power:VBUS #PWR0505
+L FHNW-Pro4E-FS19T8-3DPrinterBoard-STM32-rescue:VBUS-power #PWR0505
 U 1 1 5CC883C1
 P 3450 2350
@@
 	4000 2450 4000 2900
 $Comp
-L Power_Protection:USBLC6-2SC6 U1
+L FHNW-Pro4E-FS19T8-3DPrinterBoard-STM32-rescue:USBLC6-2SC6-Power_Protection U1
 U 1 1 5CBD8D55
 P 2950 2350
@@
 FT_TX_A
 $Comp
-L Device:C C508
+L FHNW-Pro4E-FS19T8-3DPrinterBoard-STM32-rescue:C-Device C508
 U 1 1 5D7F38AC
 P 2350 6950
@@
 $EndComp
 $Comp
-L power:GND #PWR0517
+L FHNW-Pro4E-FS19T8-3DPrinterBoard-STM32-rescue:GND-power #PWR0517
 U 1 1 5D7F38B6
 P 2350 7200
@@
 	2350 7200 2350 7100
 $Comp
-L power:+3.3V #PWR0516
+L FHNW-Pro4E-FS19T8-3DPrinterBoard-STM32-rescue:+3.3V-power #PWR0516
 U 1 1 5D7F38C2
 P 2350 6700
@@
 	1    0    0    -1
 $EndComp
+Text Notes 9450 5050 0    50   ~ 10
+YELLOW
+Text Notes 9900 5050 0    50   ~ 10
+YELLOW
+Text Notes 10350 5050 0    50   ~ 10
+YELLOW
+Text Notes 10800 5050 0    50   ~ 10
+YELLOW
+Text Notes 3650 4300 0    50   ~ 10
+100n
 $EndSCHEMATC
