File: FHNW-Pro4E-FS19T8-3DPrinterBoard-STM32.kicad_pcb (KiCad board)
At the start: 4 copper layers, 155 x 95 mm, 199 parts, among them J101 Screw_Terminal_01x02, J201 Micro_SD_Card_Det, J202 Conn_02x05_Odd_Even, J204 Conn_ARM_JTAG_SWD_10, J401 Conn_01x02, J402 Conn_01x02, J403 Screw_Terminal_01x02, J404 Conn_01x02, J405 Conn_01x02, J406 Screw_Terminal_01x02, J407 Conn_01x02, J408 Conn_01x02, J409 Conn_01x02, J410 Conn_01x02, J411 Conn_01x02, J504 USB_C_Receptacle, J601 B4B-XH-A, J602 B4B-XH-A, J603 B4B-XH-A, J604 B4B-XH-A, Q301 2N3904, Q302 2N3904, SW201 SW_Push, SW301 SW_Push, SW302 SW_Push, T401 BUK963R3-60E, T402 BUK963R3-60E, T403 BUK963R3-60E, T404 BUK963R3-60E, T405 BUK963R3-60E, U101 LM2675M-3.3, U102 LM2675M-5, U201 STM32F103ZETx, U202 NTS0104PW-Q100J, U301 ESP32-WROOM-32, U502 FT2232D, U601 TMC2660, U602 TMC2660, U603 TMC2660, U604 TMC2660, X201 SG-210STF, X501 SG5032CCN-6.000000M-HJGA3

Commit message: started with STM32 Pinout connections (Mittagspause)
Parts:
- removed D501: USBLC6-2SC6, digikey-footprints:SOT23-6L
- removed Q301, Q302: 2N3904, digikey-footprints:TO-92-3
- removed R403, R408, R412, R414: nc, Resistors_SMD:R_0603
- added C1: 33n, Capacitors_SMD:C_0603, F.Cu at (280.5, -2.56)
- added C203: 10n, Capacitors_SMD:C_0603, F.Cu at (258.6, -8.17)
- added D104: LED, LED_SMD:LED_0805_2012Metric, F.Cu at (288.0, -5.86)
- added D405: Shottky STPS1L30A, Diodes_SMD:D_SMB, F.Cu at (280.3, -13.2)
- added Q1: 2N3904, TO_SOT_Packages_SMD:SOT-23, F.Cu at (210.2, 43.2)
- added Q2: 2N3904, TO_SOT_Packages_SMD:SOT-23, F.Cu at (210.2, 38.1)
- added R102: 330R, Resistors_SMD:R_0603, F.Cu at (292.0, -6.14)
- added R213: 10k, Resistors_SMD:R_0603, F.Cu at (267.4, -14.8)
- added R214: 10k, Resistors_SMD:R_0603, F.Cu at (262.3, -8.10)
- added R215: 10k, Resistors_SMD:R_0603, F.Cu at (267.4, -12.3)
- added R216: 10k, Resistors_SMD:R_0603, F.Cu at (271.0, -14.8)
- added U1: USBLC6-2SC6, Package_TO_SOT_SMD:SOT-23-6, F.Cu at (276.1, -1.41)
- added U203: NTS0104PW-Q100J, Housings_SSOP:TSSOP-14_4.4x5mm_Pitch0.65mm, F.Cu at (261.2, -12.7)
- R207, R208: value 100k -> 10k
- moved F401 165.8 mm to (19.1, -15.2), turned to 270 degrees
- moved F402 158.3 mm to (26.0, -15.2), turned to 270 degrees
- moved T403 101.6 mm to (8.89, -12.5)
- moved R411 101.6 mm to (8.26, -5.71)
- moved J403 95.8 mm to (24.1, -27.3)
- moved J406 95.8 mm to (13.3, -27.3)
- moved R407 91.2 mm to (33.0, -5.71)
- moved T402 91.2 mm to (33.7, -12.5)
- moved U502 90.3 mm to (210.2, 61.0)
- moved J401 76.4 mm to (72.4, -29.2)
- moved R404 76.4 mm to (74.3, -9.53)
- moved T404 76.4 mm to (62.9, -16.4)
- moved J409 76.4 mm to (60.3, -29.2)
- moved R413 76.4 mm to (62.2, -9.53)
- moved T401 76.4 mm to (75.2, -16.5)
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Connections:
- net /appendix_SENSORS_POWER/ADC_Temp_Bed renamed /appendix_SENSORS_POWER/ADC_TEMP_BED
- net /appendix_SENSORS_POWER/ADC_Temp_E1 renamed /appendix_SENSORS_POWER/ADC_TEMP_E1
- net /appendix_SENSORS_POWER/ADC_Temp_MOSFET renamed /appendix_SENSORS_POWER/ADC_TEMP_PCB
- net /appendix_SENSORS_POWER/DP_Bed renamed /appendix_SENSORS_POWER/BED_ON
- net /appendix_SENSORS_POWER/DP_E1 renamed /appendix_SENSORS_POWER/E1_ON
- net /appendix_SENSORS_POWER/DP_Fan_1 renamed /appendix_SENSORS_POWER/FAN1_ON
- net /appendix_SENSORS_POWER/DP_Fan_2 renamed /appendix_SENSORS_POWER/FAN2_ON
- net /appendix_SENSORS_POWER/DP_Fan_PCB renamed /appendix_SENSORS_POWER/FAN3_ON
- net /appendix_SENSORS_POWER/SW_End_Filament renamed /appendix_SENSORS_POWER/SW_End_Filament_1
- net /appendix_SENSORS_POWER/SW_End_X_min renamed /appendix_SENSORS_POWER/SW_End_X
- net /appendix_SENSORS_POWER/SW_End_Y_min renamed /appendix_SENSORS_POWER/SW_End_Y
- net /appendix_SENSORS_POWER/SW_End_Z1_min renamed /appendix_SENSORS_POWER/SW_End_Z
- net /appendix_TMC2660_X/D_INT_TMC_STALL_X renamed /appendix_TMC2660_X/TMC_STALL_X
- net /appendix_TMC2660_X/D_TMC_CS_X renamed /appendix_TMC2660_X/TMC_CS_X
- net /appendix_TMC2660_X/D_TMC_DIR_X renamed /appendix_TMC2660_X/TMC_DIR_X
- net /appendix_TMC2660_X/D_TMC_EN_X renamed /appendix_TMC2660_X/TMC_EN_X
- net /appendix_TMC2660_X/D_TMC_STEP_X renamed /appendix_TMC2660_X/TMC_STEP_X
- net /appendix_UART_USB/RX_STM_to_TX_FTDI renamed Net-(U502-Pad24)
- net /appendix_UART_USB/TX_STM_to_RX_FTDI renamed Net-(U502-Pad23)
- net 5V renamed +5V
- net Net-(U201-Pad101) renamed /appendix_STM32F103/USART2_TX
- net Net-(U201-Pad102) renamed /appendix_STM32F103/USART2_RX
- C501 pad 1: GND -> Net-(C501-Pad1)
- C501 pad 2: Net-(C501-Pad2) -> GND
- C504 pad 1: 3.3V -> +3V3
- D502 pad 2: 3.3V -> +3V3
- D503 pad 2: 3.3V -> +3V3
- D504 pad 2: 3.3V -> +3V3
- D505 pad 2: 3.3V -> +3V3
- J201 pad 1: Net-(J201-Pad1) -> SD_DAT2
- J201 pad 10: Net-(J201-Pad10) -> SD_DETECT
- J201 pad 2: Net-(J201-Pad2) -> SD_DAT3
- J201 pad 3: Net-(J201-Pad3) -> SD_CMD
- J201 pad 4: GND -> +3V3
- J201 pad 5: Net-(J201-Pad5) -> SD_CLK
- J201 pad 6: +3V3 -> GND
- J201 pad 7: Net-(J201-Pad7) -> SD_DAT0
- J201 pad 8: Net-(J201-Pad8) -> SD_DAT1
- J201 pad 9: Net-(J201-Pad9) -> GND
- R207 pad 1: Net-(R207-Pad1) -> +3V3
- R207 pad 2: GND -> SD_DAT1
- R208 pad 1: Net-(R208-Pad1) -> +3V3
- R208 pad 2: GND -> SD_DAT0
- R302 pad 2: /appendix_ESP32/RTS_ESP32 -> /appendix_ESP32/ESP_RTS
- R303 pad 2: /appendix_ESP32/DTR_ESP32 -> /appendix_ESP32/ESP_DTR
- R501 pad 1: Net-(C501-Pad2) -> Net-(C501-Pad1)
- U201 pad 111: Net-(U201-Pad111) -> SD_DAT2
- U201 pad 112: Net-(U201-Pad112) -> SD_DAT3
- U201 pad 113: Net-(U201-Pad113) -> SD_CLK
- U201 pad 116: Net-(U201-Pad116) -> SD_CMD
- U201 pad 36: Net-(U201-Pad36) -> /appendix_ESP32/ESP_RX_STM
- U201 pad 37: Net-(U201-Pad37) -> /appendix_ESP32/ESP_TX_STM
- U201 pad 53: Net-(U201-Pad53) -> /appendix_STM32F103/STEP_Y
- U201 pad 54: Net-(U201-Pad54) -> /appendix_STM32F103/DIR_Y
- U201 pad 55: Net-(U201-Pad55) -> /appendix_STM32F103/STALL_Y
- U201 pad 56: Net-(U201-Pad56) -> /appendix_STM32F103/EN_Y
- U201 pad 57: Net-(U201-Pad57) -> /appendix_STM32F103/CS_Y
- U201 pad 74: Net-(U201-Pad74) -> /appendix_STM32F103/SPI2_SCK
- U201 pad 75: Net-(U201-Pad75) -> /appendix_STM32F103/SPI2_MISO
- U201 pad 76: Net-(U201-Pad76) -> /appendix_STM32F103/SPI2_MOSI
- U201 pad 80: Net-(U201-Pad80) -> /appendix_STM32F103/CS_Z1
- U201 pad 81: Net-(U201-Pad81) -> /appendix_STM32F103/EN_Z1
- U201 pad 82: Net-(U201-Pad82) -> /appendix_STM32F103/STALL_Z1
- U201 pad 87: Net-(U201-Pad87) -> /appendix_STM32F103/STEP_Z1
- U201 pad 88: Net-(U201-Pad88) -> /appendix_STM32F103/DIR_Z1
- U201 pad 89: Net-(U201-Pad89) -> /appendix_STM32F103/STEP_E1
- U201 pad 90: Net-(U201-Pad90) -> /appendix_STM32F103/DIR_E1
- U201 pad 91: Net-(U201-Pad91) -> /appendix_STM32F103/STALL_E1
- U201 pad 92: Net-(U201-Pad92) -> /appendix_STM32F103/EN_E1
- U201 pad 93: Net-(U201-Pad93) -> /appendix_STM32F103/CS_E1
- U201 pad 98: Net-(U201-Pad98) -> SD_DAT0
- U201 pad 99: Net-(U201-Pad99) -> SD_DAT1
- U202 pad 10: Net-(R208-Pad1) -> Net-(U202-Pad10)
- U202 pad 5: Net-(R207-Pad1) -> Net-(U202-Pad5)
- U301 pad 27: Net-(U301-Pad27) -> /appendix_ESP32/ESP_RX_STM
- U301 pad 28: Net-(U301-Pad28) -> /appendix_ESP32/ESP_TX_STM
- U301 pad 34: /appendix_ESP32/RX_ESP_to_TX_FTDI -> /appendix_ESP32/ESP_RX_USB
- U301 pad 35: /appendix_ESP32/TX_ESP_to_RX_FTDI -> /appendix_ESP32/ESP_TX_USB
- U502 pad 10: 3.3V -> +3V3
- U502 pad 14: 3.3V -> +3V3
- U502 pad 26: 3.3V -> +3V3
- U502 pad 31: 3.3V -> +3V3
- U502 pad 36: /appendix_UART_USB/DTR_ESP32 -> /appendix_ESP32/ESP_DTR
- U502 pad 38: /appendix_UART_USB/RTS_ESP32 -> /appendix_ESP32/ESP_RTS
- U502 pad 39: /appendix_UART_USB/TX_ESP_to_RX_FTDI -> /appendix_ESP32/ESP_TX_USB
- U502 pad 40: /appendix_UART_USB/RX_ESP_to_TX_FTDI -> /appendix_ESP32/ESP_RX_USB
- U502 pad 46: Net-(C501-Pad2) -> Net-(C501-Pad1)
- U502 pad 6: GND -> Net-(C1-Pad2)
- U601 pad 14: /appendix_TMC2660_X/D_SPI_MISO -> /appendix_STM32F103/SPI2_MISO
- U601 pad 15: /appendix_TMC2660_X/D_SPI_MOSI -> /appendix_STM32F103/SPI2_MOSI
- U601 pad 16: /appendix_TMC2660_X/D_SPI_SCK -> /appendix_STM32F103/SPI2_SCK
- U601 pad 18: /appendix_TMC2660_X/D_TMC_CS_Y -> /appendix_STM32F103/CS_Y
- U601 pad 19: /appendix_TMC2660_X/D_TMC_EN_Y -> /appendix_STM32F103/EN_Y
- U601 pad 38: /appendix_TMC2660_X/D_INT_TMC_STALL_Y -> /appendix_STM32F103/STALL_Y
- U601 pad 41: /appendix_TMC2660_X/D_TMC_DIR_Y -> /appendix_STM32F103/DIR_Y
- U601 pad 42: /appendix_TMC2660_X/D_TMC_STEP_Y -> /appendix_STM32F103/STEP_Y
- U602 pad 14: /appendix_TMC2660_X/D_SPI_MISO -> /appendix_STM32F103/SPI2_MISO
- U602 pad 15: /appendix_TMC2660_X/D_SPI_MOSI -> /appendix_STM32F103/SPI2_MOSI
- U602 pad 16: /appendix_TMC2660_X/D_SPI_SCK -> /appendix_STM32F103/SPI2_SCK
- U603 pad 14: /appendix_TMC2660_X/D_SPI_MISO -> /appendix_STM32F103/SPI2_MISO
- U603 pad 15: /appendix_TMC2660_X/D_SPI_MOSI -> /appendix_STM32F103/SPI2_MOSI
- U603 pad 16: /appendix_TMC2660_X/D_SPI_SCK -> /appendix_STM32F103/SPI2_SCK
- U603 pad 18: /appendix_TMC2660_X/D_TMC_CS_E1 -> /appendix_STM32F103/CS_E1
- U603 pad 19: /appendix_TMC2660_X/D_TMC_EN_E1 -> /appendix_STM32F103/EN_E1
- U603 pad 38: /appendix_TMC2660_X/D_INT_TMC_STALL_E1 -> /appendix_STM32F103/STALL_E1
- U603 pad 41: /appendix_TMC2660_X/D_TMC_DIR_E1 -> /appendix_STM32F103/DIR_E1
- U603 pad 42: /appendix_TMC2660_X/D_TMC_STEP_E1 -> /appendix_STM32F103/STEP_E1
- U604 pad 14: /appendix_TMC2660_X/D_SPI_MISO -> /appendix_STM32F103/SPI2_MISO
- U604 pad 15: /appendix_TMC2660_X/D_SPI_MOSI -> /appendix_STM32F103/SPI2_MOSI
- U604 pad 16: /appendix_TMC2660_X/D_SPI_SCK -> /appendix_STM32F103/SPI2_SCK
- U604 pad 18: /appendix_TMC2660_X/D_TMC_CS_Z1 -> /appendix_STM32F103/CS_Z1
- U604 pad 19: /appendix_TMC2660_X/D_TMC_EN_Z1 -> /appendix_STM32F103/EN_Z1
- U604 pad 38: /appendix_TMC2660_X/D_INT_TMC_STALL_Z1 -> /appendix_STM32F103/STALL_Z1
- U604 pad 41: /appendix_TMC2660_X/D_TMC_DIR_Z1 -> /appendix_STM32F103/DIR_Z1
- U604 pad 42: /appendix_TMC2660_X/D_TMC_STEP_Z1 -> /appendix_STM32F103/STEP_Z1
Routing:
- net /appendix_STM32F103/SPI2_MISO: track 0.00 -> 132.3 mm, vias 0 -> 4
- net /appendix_STM32F103/SPI2_SCK: track 0.00 -> 129.2 mm, vias 0 -> 4
- net /appendix_STM32F103/SPI2_MOSI: track 0.00 -> 124.3 mm, vias 0 -> 4
- net /appendix_TMC2660_X/D_SPI_MISO: track 93.8 -> 0.00 mm, vias 4 -> 0
- net /appendix_TMC2660_X/D_SPI_SCK: track 92.4 -> 0.00 mm, vias 4 -> 0
- net /appendix_TMC2660_X/D_SPI_MOSI: track 86.9 -> 0.00 mm, vias 4 -> 0
- net GND: track 105.6 -> 73.4 mm
- net /appendix_STM32F103/CS_E1: track 0.00 -> 32.0 mm, vias 0 -> 1
- net +24V: track 66.0 -> 35.0 mm
- net /appendix_STM32F103/EN_E1: track 0.00 -> 28.2 mm, vias 0 -> 1
- net /appendix_TMC2660_X/TMC_CS_X: track 32.3 -> 5.21 mm
- net /appendix_TMC2660_X/TMC_EN_X: track 29.6 -> 3.58 mm
- net SD_DAT0: track 0.00 -> 17.7 mm
- net Net-(J201-Pad7): track 17.7 -> 0.00 mm
- net /appendix_STM32F103/STEP_E1: track 0.00 -> 16.6 mm, vias 0 -> 1
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
Commit message: layouted FT2232 / SD card
Parts:
- added C210: 100n, Capacitors_SMD:C_0603, F.Cu at (203.1, 84.8)
- added C211: 100n, Capacitors_SMD:C_0603, F.Cu at (192.8, 84.8)
- added C212: 100n, Capacitors_SMD:C_0603, F.Cu at (203.1, 89.2)
- added C213: 100n, Capacitors_SMD:C_0603, F.Cu at (192.8, 89.2)
- J504: footprint Connector_USB:USB_C_Receptacle_GCT_USB4085 -> Connectors_USB:USB_C_Receptacle_Amphenol_12401610E4-2A
- L501: footprint Resistors_SMD:R_0805_HandSoldering -> FHNW-Pro4E-FS19T8-Library:WURTH_USB_Chocke_4PAD
- moved U203 123.0 mm to (189.1, 87.0), turned to 270 degrees
- moved R216 105.7 mm to (231.1, 83.2), turned to 180 degrees
- moved C506 103.5 mm to (205.7, 63.2), turned to 180 degrees
- moved R213 101.6 mm to (218.4, 74.3)
- moved D402 98.7 mm to (23.7, 7.62)
- moved R417 98.7 mm to (23.7, 3.81)
- moved D401 98.7 mm to (21.2, 7.62)
- moved R416 98.7 mm to (21.2, 3.81)
- moved X501 98.6 mm to (209.9, 64.3)
- moved R215 96.2 mm to (218.4, 70.5)
- moved D505 95.9 mm to (198.8, 54.0), turned to 180 degrees
- moved C203 94.2 mm to (231.1, 81.9), turned to 180 degrees
- moved U202 93.1 mm to (199.4, 87.0), turned to 270 degrees
- moved R510 92.3 mm to (201.9, 56.5), turned to 180 degrees
- moved C1 92.0 mm to (215.3, 62.4), turned to 90 degrees
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Connections:
- net /appendix_SENSORS_POWER/ADC_TEMP_BED renamed /ADC_TEMP_BED
- net /appendix_SENSORS_POWER/ADC_TEMP_E1 renamed /ADC_TEMP_E1
- net /appendix_SENSORS_POWER/ADC_TEMP_PCB renamed /ADC_TEMP_PCB
- net /appendix_SENSORS_POWER/BED_ON renamed /POWER_BED
- net /appendix_SENSORS_POWER/E1_ON renamed /POWER_E1
- net /appendix_SENSORS_POWER/FAN1_ON renamed /FAN1
- net /appendix_SENSORS_POWER/FAN2_ON renamed /FAN2
- net /appendix_SENSORS_POWER/FAN3_ON renamed /FAN3
- net /appendix_SENSORS_POWER/SW_End_Filament_1 renamed /SW_End_Filament1
- net /appendix_SENSORS_POWER/SW_End_X renamed /SW_Min_X
- net /appendix_SENSORS_POWER/SW_End_Y renamed /SW_Min_Y
- net /appendix_SENSORS_POWER/SW_End_Z renamed /SW_Min_Z
- net /appendix_STM32F103/SPI2_MISO renamed MISO
- net D_LCD_CS renamed Net-(U202-Pad4)
- net D_LCD_MOSI renamed Net-(U202-Pad3)
- net D_LCD_SCK renamed Net-(U202-Pad2)
- J202 pad 1: D_LCD_Beeper -> EXP3_LCD_Beeper
- J202 pad 2: D_LCD_Encoder_BTN -> EXP3_LCD_Encoder_BTN
- J202 pad 3: D_LCD_Encoder_B -> EXP3_LCD_Encoder_B
- J202 pad 4: D_LCD_Reset -> EXP3_LCD_Reset
- J202 pad 5: D_LCD_Encoder_A -> EXP3_LCD_Encoder_A
- J202 pad 6: Conn_LCD_SCK -> EXP3_LCD_SCK
- J202 pad 7: Conn_LCD_CS -> EXP3_LCD_CS
- J202 pad 8: Conn_LCD_MOSI -> EXP3_LCD_MOSI
- U1 pad 1: /appendix_UART_USB/USB_D_N -> /appendix_UART_USB/USB_TVS_D_N
- U1 pad 3: /appendix_UART_USB/USB_D_P -> /appendix_UART_USB/USB_TVS_D_P
- U1 pad 4: /appendix_UART_USB/USB_TVS_D_P -> /appendix_UART_USB/USB_D_P
- U1 pad 6: /appendix_UART_USB/USB_TVS_D_N -> /appendix_UART_USB/USB_D_N
- U201 pad 101: /appendix_STM32F103/USART2_TX -> /appendix_UART_USB/FT_RX_A
- U201 pad 102: /appendix_STM32F103/USART2_RX -> /appendix_UART_USB/FT_TX_A
- U201 pad 74: /appendix_STM32F103/SPI2_SCK -> SCK
- U201 pad 76: /appendix_STM32F103/SPI2_MOSI -> MOSI
- U202 pad 10: Net-(U202-Pad10) -> EXP3_LCD_Encoder_BTN
- U202 pad 11: Conn_LCD_CS -> EXP3_LCD_Reset
- U202 pad 12: Conn_LCD_MOSI -> EXP3_LCD_SCK
- U202 pad 13: Conn_LCD_SCK -> EXP3_LCD_MOSI
- U203 pad 10: Net-(U203-Pad10) -> EXP3_LCD_CS
- U203 pad 11: Net-(U203-Pad11) -> EXP3_LCD_Encoder_A
- U203 pad 12: Net-(U203-Pad12) -> EXP3_LCD_Encoder_B
- U203 pad 13: Net-(U203-Pad13) -> EXP3_LCD_Beeper
- U502 pad 23: Net-(U502-Pad23) -> /appendix_UART_USB/FT_RX_A
- U502 pad 24: Net-(U502-Pad24) -> /appendix_UART_USB/FT_TX_A
- U601 pad 15: /appendix_STM32F103/SPI2_MOSI -> SCK
- U601 pad 16: /appendix_STM32F103/SPI2_SCK -> MOSI
- U602 pad 15: /appendix_STM32F103/SPI2_MOSI -> SCK
- U602 pad 16: /appendix_STM32F103/SPI2_SCK -> MOSI
- U603 pad 15: /appendix_STM32F103/SPI2_MOSI -> SCK
- U603 pad 16: /appendix_STM32F103/SPI2_SCK -> MOSI
- U604 pad 15: /appendix_STM32F103/SPI2_MOSI -> SCK
- U604 pad 16: /appendix_STM32F103/SPI2_SCK -> MOSI
Routing:
- net MOSI: track 0.00 -> 129.2 mm, vias 0 -> 4
- net /appendix_STM32F103/SPI2_SCK: track 129.2 -> 0.00 mm, vias 4 -> 0
- net SCK: track 0.00 -> 124.3 mm, vias 0 -> 4
- net /appendix_STM32F103/SPI2_MOSI: track 124.3 -> 0.00 mm, vias 4 -> 0
- net GND: track 73.4 -> 182.8 mm, vias 72 -> 80
- net +3V3: track 25.9 -> 77.4 mm
- net +5V: track 0.00 -> 46.2 mm
- net /appendix_ESP32/ESP_RTS: track 2.92 -> 42.1 mm, vias 0 -> 2
- net /appendix_ESP32/ESP_TX_USB: track 0.00 -> 35.3 mm, vias 0 -> 2
- net /appendix_ESP32/ESP_RX_USB: track 0.00 -> 30.9 mm, vias 0 -> 2
- net /appendix_ESP32/ESP32_RESET: track 0.00 -> 25.1 mm
- net /appendix_ESP32/ESP_DTR: track 2.92 -> 27.7 mm, vias 0 -> 2
- net EXP3_LCD_MOSI: track 0.00 -> 21.2 mm
- net VBUS: track 0.00 -> 20.5 mm, vias 0 -> 3
- net EXP3_LCD_SCK: track 0.00 -> 17.6 mm
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- added copper zone on F.Cu, net +5V
- added copper zone on F.Cu, net Net-(C109-Pad1)
- added copper zone on F.Cu, net Net-(C109-Pad2)
- removed copper zone on F.Cu, net /appendix_SENSORS_POWER/Bed_pwr
- removed copper zone on F.Cu, net /appendix_SENSORS_POWER/E1_pwr
- removed copper zone on F.Cu, net /appendix_SENSORS_POWER/Fan1_pwr
- removed copper zone on F.Cu, net /appendix_SENSORS_POWER/Fan2_pwr
- removed copper zone on F.Cu, net Net-(R411-Pad1)
