File: appendix_STM32F103.sch (KiCad schematic (older format))
At the start: 40 parts, among them J201 Micro_SD_Card_Det, J202 Conn_02x05_Odd_Even, J203 Conn_02x20_Odd_Even, J204 Conn_ARM_JTAG_SWD_10, SW201 SW_Push, U201 STM32F103ZETx, U202 NTS0104PW-Q100J, U203 NTS0104PW-Q100J, X201 SG-210STF

Commit message: having issues with netclasses
Parts:
- added C214: 100n, Capacitors_SMD:C_0603, symbol Device:C
Connections:
- net +3.3VA: now also C214.1
- net +5V: no longer J203.5 (Pin_5), J203.6 (Pin_6)
- net CS_Z1: now also U201.88 (PG3); no longer U201.80 (PD11)
- net DIR_Z1: now also U201.81 (PD12); no longer U201.88 (PG3)
- net E2_ADC_TEMP: now also J203.26 (Pin_26)
- net E2_CS: now also J203.14 (Pin_14)
- net E2_EN: now also J203.20 (Pin_20)
- net E2_END_FIL: now also J203.24 (Pin_24)
- net E2_FAN1: now also J203.30 (Pin_30)
- net E2_FAN2: now also J203.32 (Pin_32)
- net E2_HOTEND: now also J203.34 (Pin_34)
- net E2_STALL: now also J203.22 (Pin_22)
- net E2_STEP: now also J203.16 (Pin_16)
- net E3_CS: now also J203.13 (Pin_13)
- net EN_Z1: now also U201.87 (PG2); no longer U201.81 (PD12)
- net ES_DIR: now also J203.18 (Pin_18)
- net FAN_EXT: now also J203.28 (Pin_28)
- net GND: now also C214.2
- net STEP_Z1: now also U201.80 (PD11); no longer U201.87 (PG2)
- net CS_X: now reaches U201.11 (PF1)
- net EN_X: now reaches U201.12 (PF2)
- net STALL_X: now reaches U201.13 (PF3)
- net DIR_X: now reaches U201.14 (PF4)
- net STEP_X: now reaches U201.15 (PF5)
- net ADC_T_BED: now reaches U201.28 (PC2)
- net ADC_T_E1: now reaches U201.29 (PC3)
- net BED_ON: now reaches U201.70 (PB11)
- net GPIO_EXT_0: now reaches J203.12 (Pin_12)
- net E3_STEP: now reaches J203.15 (Pin_15)
- net E3_DIR: now reaches J203.17 (Pin_17)
- net E3_EN: now reaches J203.19 (Pin_19)
- net E3_STALL: now reaches J203.21 (Pin_21)
- net E3_END_FIL: now reaches J203.23 (Pin_23)
- net E3_ADC_TEMP: now reaches J203.25 (Pin_25)
- net ADC_TEMP_EXT: now reaches J203.27 (Pin_27)
- net GPIO_EXT_1: now reaches J203.29 (Pin_29)
- net GPIO_EXT_2: now reaches J203.31 (Pin_31)
- net GPIO_EXT_3: now reaches J203.33 (Pin_33)
- no-connect marks 28 -> 30
Other:
- note added: "RC_ für ADC\n"
- note added: "TVS Diode"
- note removed: "double check pinout with footprint!!!"
Changed lines of the file:
@@
 Text HLabel 7900 3700 0    50   Input ~ 0
 CS_Y
-Text HLabel 7900 3800 0    50   Input ~ 0
+Text HLabel 10900 8100 2    50   Input ~ 0
 STEP_Z1
-Text HLabel 7900 3900 0    50   Input ~ 0
-DIR_Z1
 Text HLabel 7900 4000 0    50   Input ~ 0
 STEP_E1
@@
 Text HLabel 7900 6800 0    50   Input ~ 0
 STALL_Y
-Text HLabel 10900 8100 2    50   Input ~ 0
-CS_Z1
-Text HLabel 10900 8200 2    50   Input ~ 0
-EN_Z1
-Text HLabel 10900 8300 2    50   Input ~ 0
-STALL_Z1
-Text Notes 14200 3550 0    50   ~ 0
-double check pinout with footprint!!!
 Wire Wire Line
 	14850 5100 14650 5100
@@
 Wire Wire Line
 	6500 9250 6600 9250
-$Comp
-L power:+5V #PWR0172
-U 1 1 5D3333A6
-P 7200 9150
-F 0 "#PWR0172" H 7200 9000 50  0001 C CNN
-F 1 "+5V" V 7200 9350 50  0000 C CNN
-F 2 "" H 7200 9150 50  0001 C CNN
-F 3 "" H 7200 9150 50  0001 C CNN
-	1    7200 9150
-	0    1    1    0
-$EndComp
-$Comp
-L power:+5V #PWR0173
-U 1 1 5D334323
-P 6500 9150
-F 0 "#PWR0173" H 6500 9000 50  0001 C CNN
-F 1 "+5V" V 6500 9350 50  0000 C CNN
-F 2 "" H 6500 9150 50  0001 C CNN
-F 3 "" H 6500 9150 50  0001 C CNN
-	1    6500 9150
-	0    -1   -1   0
-$EndComp
 Wire Wire Line
 	6500 9150 6600 9150
@@
 Wire Wire Line
 	7100 9350 7200 9350
-Text GLabel 7200 9450 2    50   Input ~ 0
-E3_CS
 Text GLabel 7200 9550 2    50   Input ~ 0
 E2_CS
@@
 U 1 1 5CDCD7F7
 P 14100 8500
-F 0 "R217" V 14200 8550 50  0000 C CNN
+F 0 "R217" V 14200 8500 50  0000 C CNN
 F 1 "200R" V 14100 8500 50  0000 C CNN
 F 2 "Resistors_SMD:R_0603" V 14030 8500 50  0001 C CNN
@@
 	1    0    0    -1
 $EndComp
+Text Notes 7950 10350 0    50   ~ 0
+RC_ für ADC\n
+Text Notes 13950 8100 0    50   ~ 0
+TVS Diode
+Text HLabel 10900 8200 2    50   Input ~ 0
+DIR_Z1
+Text HLabel 7900 3800 0    50   Input ~ 0
+EN_Z1
+Text HLabel 7900 3900 0    50   Input ~ 0
+CS_Z1
+Text HLabel 10900 8300 2    50   Input ~ 0
+STALL_Z1
+Text HLabel 7900 5800 0    50   Input ~ 0
+STEP_X
+Text HLabel 7900 5700 0    50   Input ~ 0
+DIR_X
+Text HLabel 7900 5600 0    50   Input ~ 0
+STALL_X
+Text HLabel 7900 5500 0    50   Input ~ 0
+EN_X
+Text HLabel 7900 5400 0    50   Input ~ 0
+CS_X
+Wire Wire Line
+	7900 5600 8100 5600
+Wire Wire Line
+	8100 5700 7900 5700
+Wire Wire Line
+	7900 5400 8100 5400
+Wire Wire Line
+	8100 5500 7900 5500
+Wire Wire Line
+	7900 5800 8100 5800
+$Comp
+L Device:C C214
+U 1 1 5CE6D10B
+P 5300 10550
+F 0 "C214" H 5415 10596 50  0000 L CNN
+F 1 "100n" H 5415 10505 50  0000 L CNN
+F 2 "Capacitors_SMD:C_0603" H 5338 10400 50  0001 C CNN
+F 3 "~" H 5300 10550 50  0001 C CNN
+	1    5300 10550
+	1    0    0    -1
+$EndComp
+$Comp
+L power:GND #PWR0235
+U 1 1 5CE6D115
+P 5300 10800
+F 0 "#PWR0235" H 5300 10550 50  0001 C CNN
+F 1 "GND" H 5305 10627 50  0000 C CNN
+F 2 "" H 5300 10800 50  0001 C CNN
+F 3 "" H 5300 10800 50  0001 C CNN
+	1    5300 10800
+	1    0    0    -1
+$EndComp
+Wire Wire Line
+	5300 10400 5300 10300
+Wire Wire Line
+	5300 10800 5300 10700
+$Comp
+L power:+3.3VA #PWR?
+U 1 1 5CE9FD57
+P 5300 10300
+AR Path="/5CE9FD57" Ref="#PWR?"  Part="1"
+AR Path="/5CA3954A/5CE9FD57" Ref="#PWR0234"  Part="1"
+F 0 "#PWR0234" H 5300 10150 50  0001 C CNN
+F 1 "+3.3VA" H 5315 10473 50  0000 C CNN
+F 2 "" H 5300 10300 50  0001 C CNN
+F 3 "" H 5300 10300 50  0001 C CNN
+	1    5300 10300
+	1    0    0    -1
+$EndComp
+Text HLabel 10900 5600 2    50   Input ~ 0
+ADC_T_E1
+Text HLabel 10900 5500 2    50   Input ~ 0
+ADC_T_BED
+Wire Wire Line
+	10900 5500 10700 5500
+Wire Wire Line
+	10700 5600 10900 5600
+Text HLabel 10850 4700 2    50   Input ~ 0
+BED_ON
+Text HLabel 10900 4400 2    50   Input ~ 0
+E1_ON
+Wire Wire Line
+	10850 4700 10700 4700
+Wire Wire Line
+	10850 4600 10700 4600
+Text GLabel 6500 9550 0    50   Input ~ 0
+E3_CS
+Text GLabel 6500 9650 0    50   Input ~ 0
+E3_STEP
+Text GLabel 6500 9750 0    50   Input ~ 0
+E3_DIR
+Text GLabel 6500 9850 0    50   Input ~ 0
+E3_EN
+Text GLabel 6500 9950 0    50   Input ~ 0
+E3_STALL
+Text GLabel 6500 10050 0    50   Input ~ 0
+E3_END_FIL
+Text GLabel 6500 10150 0    50   Input ~ 0
+E3_ADC_TEMP
+Text GLabel 6500 10250 0    50   Input ~ 0
+ADC_TEMP_EXT
+Text GLabel 6500 10350 0    50   Input ~ 0
+GPIO_EXT_1
+Text GLabel 6500 10450 0    50   Input ~ 0
+GPIO_EXT_2
+Text GLabel 6500 10550 0    50   Input ~ 0
+GPIO_EXT_3
+Text GLabel 7200 9450 2    50   Input ~ 0
+GPIO_EXT_0
+Wire Wire Line
+	6500 9650 6600 9650
+Wire Wire Line
+	6500 9550 6600 9550
+Wire Wire Line
+	6500 9750 6600 9750
+Wire Wire Line
+	6600 9850 6500 9850
+Wire Wire Line
+	6500 10050 6600 10050
+Wire Wire Line
+	6500 9950 6600 9950
+Wire Wire Line
+	6500 10150 6600 10150
+Wire Wire Line
+	6600 10250 6500 10250
+Wire Wire Line
+	6500 10450 6600 10450
+Wire Wire Line
+	6500 10350 6600 10350
+Wire Wire Line
+	6500 10550 6600 10550
+Wire Wire Line
+	7200 9450 7100 9450
+Wire Wire Line
+	7100 9650 7200 9650
+Wire Wire Line
+	7100 9550 7200 9550
+Wire Wire Line
+	7100 9750 7200 9750
+Wire Wire Line
+	7200 9850 7100 9850
+Wire Wire Line
+	7100 10050 7200 10050
+Wire Wire Line
+	7100 9950 7200 9950
+Wire Wire Line
+	7100 10150 7200 10150
+Wire Wire Line
+	7200 10250 7100 10250
+Wire Wire Line
+	7100 10450 7200 10450
+Wire Wire Line
+	7100 10350 7200 10350
+Wire Wire Line
+	7100 10550 7200 10550
+NoConn ~ 7200 9150
+NoConn ~ 6500 9150
 $EndSCHEMATC
