File: appendix_STM32F103.sch (KiCad schematic (older format))
At the start: 41 parts, among them J201 Micro_SD_Card_Det, J202 Conn_02x05_Odd_Even, J203 Conn_02x20_Odd_Even, J204 Conn_ARM_JTAG_SWD_10, SW201 SW_Push, U201 STM32F103ZETx, U202 NTS0104PW-Q100J, U203 NTS0104PW-Q100J, X201 SG-210STF

Commit message: first layout draft without 40pin
Connections:
- net +3V3: now also U202.8 (OE), U203.8 (OE)
- net +5V: no longer U202.8 (OE), U203.8 (OE)
- net ADC_T_BED: now also U201.29 (PC3); no longer U201.28 (PC2)
- net ADC_T_E1: now also U201.28 (PC2); no longer U201.29 (PC3)
- net CS_X: now also U201.50 (PF12); no longer U201.11 (PF1)
- net DIR_X: now also U201.42 (PA6); no longer U201.14 (PF4)
- net E1_ON: now also U201.69 (PB10)
- net EN_X: now also U201.49 (PF11); no longer U201.12 (PF2)
- net STALL_X: now also U201.43 (PA7); no longer U201.13 (PF3)
- net STEP_X: now also U201.41 (PA5); no longer U201.15 (PF5)
- net USART1_RX: now also U201.102 (PA10); no longer U201.37 (PA3)
- net USART1_TX: now also U201.101 (PA9); no longer U201.36 (PA2)
- net USART2_RX: now also U201.37 (PA3); no longer U201.102 (PA10)
- net USART2_TX: now also U201.36 (PA2); no longer U201.101 (PA9)
- net SW_Min_Filament1: now reaches U201.3 (PE4)
- net ADC_T_PCB: now reaches U201.35 (PA1)
- net SW_Min_Z1: now reaches U201.4 (PE5)
- new net FAN1: U201.13 (PF3)
- new net FAN2: U201.14 (PF4)
- new net FAN3: U201.15 (PF5)
- new net SW_Min_X: U201.11 (PF1)
- new net SW_Min_Y: U201.12 (PF2)
Changed lines of the file:
@@
 	14650 5400 14800 5400
-$Comp
-L power:+5V #PWR04
-U 1 1 5CBEBF25
-P 14800 5350
-F 0 "#PWR04" H 14800 5200 50  0001 C CNN
-F 1 "+5V" H 14815 5523 50  0000 C CNN
-F 2 "" H 14800 5350 50  0001 C CNN
-F 3 "" H 14800 5350 50  0001 C CNN
-	1    14800 5350
-	1    0    0    -1
-$EndComp
 $Comp
 L power:+5V #PWR03
@@
 Wire Wire Line
 	14650 6800 14800 6800
-$Comp
-L power:+5V #PWR0224
-U 1 1 5CC4D210
-P 14800 6750
-F 0 "#PWR0224" H 14800 6600 50  0001 C CNN
-F 1 "+5V" H 14815 6923 50  0000 C CNN
-F 2 "" H 14800 6750 50  0001 C CNN
-F 3 "" H 14800 6750 50  0001 C CNN
-	1    14800 6750
-	1    0    0    -1
-$EndComp
 $Comp
 L power:+5V #PWR0223
@@
 Text Notes 8550 6850 0    50   ~ 0
 INT
+Text HLabel 10850 2800 2    50   Input ~ 0
+USART1_TX
+Text HLabel 10850 2900 2    50   Input ~ 0
+USART1_RX
 Text HLabel 10850 2100 2    50   Input ~ 0
-USART1_TX
+USART2_TX
 Text HLabel 10850 2200 2    50   Input ~ 0
-USART1_RX
-Text HLabel 10850 2800 2    50   Input ~ 0
-USART2_TX
-Text HLabel 10850 2900 2    50   Input ~ 0
 USART2_RX
 Text HLabel 11750 4800 1    50   Input ~ 0
@@
 Text HLabel 10900 8300 2    50   Input ~ 0
 STALL_Z1
-Text HLabel 7900 5800 0    50   Input ~ 0
+Text HLabel 10850 2400 2    50   Input ~ 0
 STEP_X
-Text HLabel 7900 5700 0    50   Input ~ 0
+Text HLabel 10850 2500 2    50   Input ~ 0
 DIR_X
-Text HLabel 7900 5600 0    50   Input ~ 0
+Text HLabel 10850 2600 2    50   Input ~ 0
 STALL_X
-Text HLabel 7900 5500 0    50   Input ~ 0
+Text HLabel 7900 6400 0    50   Input ~ 0
 EN_X
-Text HLabel 7900 5400 0    50   Input ~ 0
+Text HLabel 7900 6500 0    50   Input ~ 0
 CS_X
-Wire Wire Line
-	7900 5600 8100 5600
-Wire Wire Line
-	8100 5700 7900 5700
-Wire Wire Line
-	7900 5400 8100 5400
-Wire Wire Line
-	8100 5500 7900 5500
-Wire Wire Line
-	7900 5800 8100 5800
 $Comp
 L Device:C C214
@@
 	1    0    0    -1
 $EndComp
+Text HLabel 10900 5500 2    50   Input ~ 0
+ADC_T_E1
 Text HLabel 10900 5600 2    50   Input ~ 0
-ADC_T_E1
-Text HLabel 10900 5500 2    50   Input ~ 0
 ADC_T_BED
 Wire Wire Line
@@
 Text HLabel 10850 4700 2    50   Input ~ 0
 BED_ON
-Text HLabel 10900 4400 2    50   Input ~ 0
+Text HLabel 10850 4600 2    50   Input ~ 0
 E1_ON
 Wire Wire Line
@@
 NoConn ~ 7200 9150
 NoConn ~ 6500 9150
+$Comp
+L power:+3.3V #PWR0173
+U 1 1 5CD063D1
+P 14800 5350
+F 0 "#PWR0173" H 14800 5200 50  0001 C CNN
+F 1 "+3.3V" H 14800 5500 50  0000 C CNN
+F 2 "" H 14800 5350 50  0001 C CNN
+F 3 "" H 14800 5350 50  0001 C CNN
+	1    14800 5350
+	1    0    0    -1
+$EndComp
+$Comp
+L power:+3.3V #PWR0187
+U 1 1 5CD069D4
+P 14800 6750
+F 0 "#PWR0187" H 14800 6600 50  0001 C CNN
+F 1 "+3.3V" H 14800 6900 50  0000 C CNN
+F 2 "" H 14800 6750 50  0001 C CNN
+F 3 "" H 14800 6750 50  0001 C CNN
+	1    14800 6750
+	1    0    0    -1
+$EndComp
+Wire Wire Line
+	10850 2400 10700 2400
+Wire Wire Line
+	10850 2500 10700 2500
+Wire Wire Line
+	10850 2600 10700 2600
+Wire Wire Line
+	7900 6500 8100 6500
+Wire Wire Line
+	7900 6400 8100 6400
+Text HLabel 7900 5600 0    50   Input ~ 0
+FAN1
+Text HLabel 7900 5700 0    50   Input ~ 0
+FAN2
+Text HLabel 7900 5800 0    50   Input ~ 0
+FAN3
+Wire Wire Line
+	7900 5800 8100 5800
+Wire Wire Line
+	7900 5700 8100 5700
+Wire Wire Line
+	7900 5600 8100 5600
+Text HLabel 10850 2000 2    50   Input ~ 0
+ADC_T_PCB
+Wire Wire Line
+	10850 2000 10700 2000
+Text HLabel 7900 5400 0    50   Input ~ 0
+SW_Min_X
+Text HLabel 7900 5500 0    50   Input ~ 0
+SW_Min_Y
+Text HLabel 7900 7500 0    50   Input ~ 0
+SW_Min_Z1
+Text HLabel 7900 7400 0    50   Input ~ 0
+SW_Min_Filament1
+Wire Wire Line
+	7900 7400 8100 7400
+Wire Wire Line
+	8100 7500 7900 7500
+Wire Wire Line
+	7900 5400 8100 5400
+Wire Wire Line
+	8100 5500 7900 5500
 $EndSCHEMATC

Commit message: user LED + fixes in Layout
Parts:
- added D202, D203: LED, LED_SMD:LED_0805_2012Metric, symbol Device:LED
- added R218, R219: 330R, Resistors_SMD:R_0603, symbol Device:R
Connections:
- net GND: now also D201.1 (K), D202.1 (K), D203.1 (K)
- net MOSI: now also U202.2 (A1)
- net SCK: now also U202.3 (A2)
- net SD_DETECT: now also U201.103 (PA11)
- net LCD_ENC_BTN: now reaches U201.1 (PE2)
- net LCD_ENC_BTN: now also U202.5 (A4)
- net LED_Marlin: now reaches U201.104 (PA12)
- net LED_Marlin: now also R219.1
- net LCD_CS: now reaches U201.139 (PB8)
- net LCD_CS: now also U203.5 (A4)
- net LCD_ENC_B: now reaches U201.140 (PB9)
- net LCD_ENC_B: now also U203.4 (A3)
- net LCD_ENC_A: now reaches U201.141 (PE0)
- net LCD_ENC_A: now also U203.3 (A2)
- net LCD_BUZZER: now reaches U201.142 (PE1)
- net LCD_BUZZER: now also U203.2 (A1)
- net LED_USER_1: now reaches U201.45 (PC5)
- net LED_USER_1: now also R202.1
- net LED_USER_2: now reaches U201.46 (PB0)
- net LED_USER_2: now also R218.1
- net LCD_Reset: now reaches U202.4 (A3)
- new net: D202.2 (A), R218.2
- new net: D203.2 (A), R219.2
Other:
- moved on the sheet: D201, R202
Changed lines of the file:
@@
 Text HLabel 10850 2200 2    50   Input ~ 0
 USART2_RX
-Text HLabel 11750 4800 1    50   Input ~ 0
+Text HLabel 11550 4800 1    50   Input ~ 0
 SPI2_SCK
 Text HLabel 11650 4800 1    50   Input ~ 0
 SPI2_MISO
-Text HLabel 11550 4800 1    50   Input ~ 0
+Text HLabel 11750 4800 1    50   Input ~ 0
 SPI2_MOSI
 Text HLabel 7900 3600 0    50   Input ~ 0
@@
 L Device:R R202
 U 1 1 5CDABFCE
-P 3350 4400
-F 0 "R202" H 3420 4446 50  0000 L CNN
-F 1 "330R" H 3420 4355 50  0000 L CNN
-F 2 "Resistors_SMD:R_0603" V 3280 4400 50  0001 C CNN
-F 3 "~" H 3350 4400 50  0001 C CNN
-	1    3350 4400
+P 950 4700
+F 0 "R202" H 1020 4746 50  0000 L CNN
+F 1 "330R" H 1020 4655 50  0000 L CNN
+F 2 "Resistors_SMD:R_0603" V 880 4700 50  0001 C CNN
+F 3 "~" H 950 4700 50  0001 C CNN
+	1    950  4700
 	1    0    0    -1
 $EndComp
@@
 L Device:LED D201
 U 1 1 5CDABFD4
-P 3350 4800
-F 0 "D201" V 3389 4683 50  0000 R CNN
-F 1 "LED" V 3298 4683 50  0000 R CNN
-F 2 "LED_SMD:LED_0805_2012Metric" H 3350 4800 50  0001 C CNN
-F 3 "~" H 3350 4800 50  0001 C CNN
-	1    3350 4800
+P 950 5100
+F 0 "D201" V 989 4983 50  0000 R CNN
+F 1 "LED" V 898 4983 50  0000 R CNN
+F 2 "LED_SMD:LED_0805_2012Metric" H 950 5100 50  0001 C CNN
+F 3 "~" H 950 5100 50  0001 C CNN
+	1    950  5100
 	0    -1   -1   0
 $EndComp
 Wire Wire Line
-	3350 4550 3350 4650
+	950  4850 950  4950
 $Comp
 L Connector_Generic:Conn_02x20_Odd_Even J203
@@
 Wire Wire Line
 	8100 5500 7900 5500
+Text GLabel 13450 4900 0    50   Input ~ 0
+SCK
+Text GLabel 13450 4800 0    50   Input ~ 0
+MOSI
+Text GLabel 13450 5000 0    50   Input ~ 0
+LCD_Reset
+Text GLabel 13450 5100 0    50   Input ~ 0
+LCD_ENC_BTN
+Text GLabel 13450 6200 0    50   Input ~ 0
+LCD_BUZZER
+Text GLabel 13450 6300 0    50   Input ~ 0
+LCD_ENC_A
+Text GLabel 13450 6400 0    50   Input ~ 0
+LCD_ENC_B
+Text GLabel 13450 6500 0    50   Input ~ 0
+LCD_CS
+Text GLabel 7900 7200 0    50   Input ~ 0
+LCD_ENC_BTN
+Wire Wire Line
+	8100 7200 7900 7200
+Text GLabel 7900 7100 0    50   Input ~ 0
+LCD_BUZZER
+Text GLabel 7900 7000 0    50   Input ~ 0
+LCD_ENC_A
+Text GLabel 10850 4500 2    50   Input ~ 0
+LCD_ENC_B
+Text GLabel 10850 4400 2    50   Input ~ 0
+LCD_CS
+Wire Wire Line
+	10850 4400 10700 4400
+Wire Wire Line
+	10700 4500 10850 4500
+Wire Wire Line
+	7900 7000 8100 7000
+Wire Wire Line
+	8100 7100 7900 7100
+Text GLabel 10850 3000 2    50   Input ~ 0
+SD_DETECT
+Wire Wire Line
+	10850 3000 10700 3000
+$Comp
+L Device:R R218
+U 1 1 5CEF3625
+P 1350 4700
+F 0 "R218" H 1420 4746 50  0000 L CNN
+F 1 "330R" H 1420 4655 50  0000 L CNN
+F 2 "Resistors_SMD:R_0603" V 1280 4700 50  0001 C CNN
+F 3 "~" H 1350 4700 50  0001 C CNN
+	1    1350 4700
+	1    0    0    -1
+$EndComp
+$Comp
+L Device:LED D202
+U 1 1 5CEF362F
+P 1350 5100
+F 0 "D202" V 1389 4983 50  0000 R CNN
+F 1 "LED" V 1298 4983 50  0000 R CNN
+F 2 "LED_SMD:LED_0805_2012Metric" H 1350 5100 50  0001 C CNN
+F 3 "~" H 1350 5100 50  0001 C CNN
+	1    1350 5100
+	0    -1   -1   0
+$EndComp
+Wire Wire Line
+	1350 4850 1350 4950
+$Comp
+L Device:R R219
+U 1 1 5CF13CB8
+P 1750 4700
+F 0 "R219" H 1820 4746 50  0000 L CNN
+F 1 "330R" H 1820 4655 50  0000 L CNN
+F 2 "Resistors_SMD:R_0603" V 1680 4700 50  0001 C CNN
+F 3 "~" H 1750 4700 50  0001 C CNN
+	1    1750 4700
+	1    0    0    -1
+$EndComp
+$Comp
+L Device:LED D203
+U 1 1 5CF13CC2
+P 1750 5100
+F 0 "D203" V 1789 4983 50  0000 R CNN
+F 1 "LED" V 1698 4983 50  0000 R CNN
+F 2 "LED_SMD:LED_0805_2012Metric" H 1750 5100 50  0001 C CNN
+F 3 "~" H 1750 5100 50  0001 C CNN
+	1    1750 5100
+	0    -1   -1   0
+$EndComp
+Wire Wire Line
+	1750 4850 1750 4950
+$Comp
+L power:GND #PWR0194
+U 1 1 5CF54C9D
+P 950 5350
+F 0 "#PWR0194" H 950 5100 50  0001 C CNN
+F 1 "GND" H 955 5177 50  0000 C CNN
+F 2 "" H 950 5350 50  0001 C CNN
+F 3 "" H 950 5350 50  0001 C CNN
+	1    950  5350
+	1    0    0    -1
+$EndComp
+Wire Wire Line
+	950  5350 950  5250
+$Comp
+L power:GND #PWR0198
+U 1 1 5CF75AD3
+P 1350 5350
+F 0 "#PWR0198" H 1350 5100 50  0001 C CNN
+F 1 "GND" H 1355 5177 50  0000 C CNN
+F 2 "" H 1350 5350 50  0001 C CNN
+F 3 "" H 1350 5350 50  0001 C CNN
+	1    1350 5350
+	1    0    0    -1
+$EndComp
+Wire Wire Line
+	1350 5350 1350 5250
+$Comp
+L power:GND #PWR0199
+U 1 1 5CF96A3E
+P 1750 5350
+F 0 "#PWR0199" H 1750 5100 50  0001 C CNN
+F 1 "GND" H 1755 5177 50  0000 C CNN
+F 2 "" H 1750 5350 50  0001 C CNN
+F 3 "" H 1750 5350 50  0001 C CNN
+	1    1750 5350
+	1    0    0    -1
+$EndComp
+Wire Wire Line
+	1750 5350 1750 5250
+Text GLabel 1900 4400 2    50   Input ~ 0
+LED_Marlin
+Wire Wire Line
+	1900 4400 1750 4400
+Wire Wire Line
+	1750 4400 1750 4550
+Text GLabel 1900 4200 2    50   Input ~ 0
+LED_USER_2
+Text GLabel 1900 4000 2    50   Input ~ 0
+LED_USER_1
+Wire Wire Line
+	1900 4200 1350 4200
+Wire Wire Line
+	1350 4200 1350 4550
+Wire Wire Line
+	1900 4000 950  4000
+Wire Wire Line
+	950  4000 950  4550
+Text GLabel 10900 5800 2    50   Input ~ 0
+LED_USER_1
+Wire Wire Line
+	10900 5800 10700 5800
+Text GLabel 10850 3600 2    50   Input ~ 0
+LED_USER_2
+Wire Wire Line
+	10850 3600 10700 3600
+Text GLabel 10850 3100 2    50   Input ~ 0
+LED_Marlin
+Wire Wire Line
+	10850 3100 10700 3100
 $EndSCHEMATC

Commit message: TVS protection, BOOT1 pin, user BTN
Parts:
- added C215, C216, C220, C221: 100n, Capacitors_SMD:C_0603, symbol Device:C
- added C217, C218, C219: 10u, Capacitors_SMD:C_1210, symbol Device:CP
- added D204, D206: BAT54C, Package_TO_SOT_SMD:SOT-23, symbol Diode:BAT54C
- added D205, D207: BAT54A, Package_TO_SOT_SMD:SOT-23, symbol Diode:BAT54A
- added D208: BAT54S, Package_TO_SOT_SMD:SOT-23, symbol Diode:BAT54S
- added R225, R227, R229: 0R, Resistors_SMD:R_0603, symbol Device:R
- added R230, R231, R232, R233, R234, R236, R237: 10k, Resistors_SMD:R_0603, symbol Device:R
- added SW202, SW203: SW_Push, Buttons_Switches_SMD:SW_SPST_KMR2, symbol Switch:SW_Push
- C202, C203: value 10n -> 100n
- C214: value 100n -> 10n
- J204: footprint Connector_PinHeader_1.27mm:PinHeader_2x05_P1.27mm_Vertical -> Connector_PinHeader_1.27mm:PinHeader_2x05_P1.27mm_Vertical_SMD
- R209, R210, R211, R212, R217: value 200R -> 100R
- SW201: footprint Button_Switch_SMD:SW_SPST_KMR2 -> Buttons_Switches_SMD:SW_SPST_KMR2
Connections:
- net +3.3VA: now also C217.1
- net +3V3: now also C218.1, C219.1, C220.1, C221.1, D204.3, D206.3, D208.2, R230.1, R231.1, R233.1, R234.1
- net GND: now also C215.2, C216.2, C217.2, C218.2, C219.2, C220.2, C221.2, D205.3, D207.3, D208.1, R232.1, R236.2, R237.2, SW202.1, SW203.1
- net JTAG_RESET: now also D208.3
- net JTAG_TCK_SWCLK: now also D204.1, D205.2
- net JTAG_TDI: now also D206.1, D207.2
- net JTAG_TDO_SWO: now also D206.2, D207.1
- net JTAG_TMS_SWDIO: now also D204.2, D205.1
- net JTAG_TRST: now also R229.2; no longer U201.134 (PB4)
- net STM_BOOT1: now also R232.2, R236.1; no longer U201.138 (BOOT0)
- net USART1_RX: now also R230.2
- net USART1_TX: now also R231.2
- net BTN_USER_1: now reaches U201.96 (PC6)
- net BTN_USER_1: now also C215.1, R233.2, SW202.2
- net BTN_USER_2: now reaches U201.97 (PC7)
- net BTN_USER_2: now also C216.1, R234.2, SW203.2
- new net NRST: R227.2, U201.134 (PB4)
- new net STM32_BOOT_0: R225.1, R237.1
- new net STM32_NRST: R227.1, R229.1
- new net STM_BOOT0: R225.2, U201.138 (BOOT0)
Other:
- note added: "JTAG"
- note added: "VDD3 (Pin 144)"
- note removed: "Layout Datasheet p.1\nhttps://support.epson.biz/td/api/doc_check.php?dl=brief_SG-210STF&lang=en\n"
- note removed: "RC_ für ADC\n"
- note removed: "TODO \nreset review by Dominik"
- note removed: "TVS Diode"
- moved on the sheet: C201, C202, C210, C211, C212, C213, C214, J203, J204, R201, R203, R204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

Commit message: finished up for final review
Parts:
- removed C221: 100n, Capacitors_SMD:C_0603, symbol Device:C
- removed R225: 0R, Resistors_SMD:R_0603, symbol Device:R
- removed R232: 10k, Resistors_SMD:R_0603, symbol Device:R
- added R220, R221: 0R, Resistors_SMD:R_0603, symbol Device:R
Connections:
- net ES_DIR is gone; now on net E2_DIR: J203.18 (Pin_18)
- net ADC_TEMP_EXT: now also U201.21 (PF9)
- net E2_ADC_TEMP: now also U201.22 (PF10)
- net E2_CS: now also U201.78 (PD9)
- net E2_EN: now also U201.125 (PG10)
- net E2_END_FIL: now also U201.129 (PG14)
- net E2_FAN1: now also U201.67 (PE14)
- net E2_FAN2: now also U201.65 (PE12)
- net E2_HOTEND: now also U201.63 (PE10)
- net E2_STALL: now also U201.126 (PG11)
- net E2_STEP: now also U201.85 (PD14)
- net E3_ADC_TEMP: now also U201.20 (PF8)
- net E3_CS: now also U201.79 (PD10)
- net E3_DIR: now also U201.124 (PG9)
- net E3_EN: now also U201.128 (PG13)
- net E3_END_FIL: now also U201.10 (PF0)
- net E3_STALL: now also U201.127 (PG12)
- net E3_STEP: now also U201.114 (PD0)
- net FAN_EXT: now also U201.68 (PE15)
- net GPIO_EXT_0: now also U201.77 (PD8)
- net GPIO_EXT_1: now also U201.66 (PE13)
- net GPIO_EXT_2: now also U201.64 (PE11)
- net GPIO_EXT_3: now also U201.60 (PE9)
- net JTAG_RESET: now also R227.2, R229.2, R220.2
- net JTAG_TRST: now also R227.1, U201.134 (PB4); no longer R229.2
- net LCD_ENC_A: now also U201.140 (PB9), U203.4 (A3); no longer U201.141 (PE0), U203.3 (A2)
- net LCD_ENC_B: now also U201.141 (PE0), U203.3 (A2); no longer U201.140 (PB9), U203.4 (A3)
- net LCD_Reset: now also R220.1
- net SERVO_1: now also U201.122 (PD6)
- net SERVO_2: now also U201.123 (PD7)
- net STM32_BOOT_0: now also R221.1; no longer R237.1
- net STM32_NRST: no longer R227.1
- net STM_BOOT0: now also R237.1, R221.2
- net E2_DIR: now reaches U201.115 (PD1)
- removed net NRST: R227.2, U201.134 (PB4)
- no-connect marks 30 -> 34
Other:
- moved on the sheet: C201, C215, C216, D201, D202, D203, D204, D205, D206, D207, D208, J204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

Commit message: fixed minor layout stuff with mueller
Parts:
- added R222: 0R, Resistors_SMD:R_0603, symbol Device:R
- C217: value 10u -> 1u
Connections:
- net +3.3VA: now also U201.32 (VREF+)
- net GND: now also U201.31 (VREF-)
- net LCD_Reset: now also R222.1
- net at U201.2 (PE3): now also R222.2
- no-connect marks 34 -> 31
Changed lines of the file:
@@
 AR Path="/5CA3954A/5CEED6D0" Ref="C217"  Part="1"
 F 0 "C217" H 5468 10596 50  0000 L CNN
-F 1 "10u" H 5468 10505 50  0000 L CNN
+F 1 "1u" H 5468 10505 50  0000 L CNN
 F 2 "Capacitors_SMD:C_1210" H 5388 10400 50  0001 C CNN
 F 3 "~" H 5350 10550 50  0001 C CNN
@@
 Wire Wire Line
 	6900 7900 7100 7900
-NoConn ~ 7100 2300
-NoConn ~ 7100 2400
 NoConn ~ 9700 2300
 NoConn ~ 9700 1900
@@
 NoConn ~ 9700 6800
 NoConn ~ 7100 6000
-NoConn ~ 7100 7300
 NoConn ~ 9700 7300
 NoConn ~ 7100 7600
@@
 Wire Wire Line
 	7100 4600 6900 4600
+Text GLabel 5750 7300 0    50   Input ~ 0
+LCD_Reset
+$Comp
+L Device:R R222
+U 1 1 5CCE79DA
+P 6100 7300
+F 0 "R222" V 6200 7300 50  0000 C CNN
+F 1 "0R" V 6100 7300 50  0000 C CNN
+F 2 "Resistors_SMD:R_0603" V 6030 7300 50  0001 C CNN
+F 3 "~" H 6100 7300 50  0001 C CNN
+	1    6100 7300
+	0    -1   -1   0
+$EndComp
+Wire Wire Line
+	5950 7300 5750 7300
+Wire Wire Line
+	7100 7300 6250 7300
+$Comp
+L power:+3.3VA #PWR0267
+U 1 1 5CDF6C38
+P 6950 2300
+F 0 "#PWR0267" H 6950 2150 50  0001 C CNN
+F 1 "+3.3VA" V 6950 2600 50  0000 C CNN
+F 2 "" H 6950 2300 50  0001 C CNN
+F 3 "" H 6950 2300 50  0001 C CNN
+	1    6950 2300
+	0    -1   -1   0
+$EndComp
+Wire Wire Line
+	7100 2300 6950 2300
+$Comp
+L power:GND #PWR0268
+U 1 1 5CE3885D
+P 7050 2400
+F 0 "#PWR0268" H 7050 2150 50  0001 C CNN
+F 1 "GND" V 7050 2150 50  0000 C CNN
+F 2 "" H 7050 2400 50  0001 C CNN
+F 3 "" H 7050 2400 50  0001 C CNN
+	1    7050 2400
+	0    1    1    0
+$EndComp
+Wire Wire Line
+	7050 2400 7100 2400
 $EndSCHEMATC
