File: appendix_SENSORS_POWER.sch (KiCad schematic (older format))
At the start: 59 parts, among them J401 Conn_01x02, J402 Conn_01x02, J403 Screw_Terminal_01x04, J404 Conn_01x02, J405 Conn_01x02, J407 Conn_01x02, J408 Conn_01x02, J409 Conn_01x02, J410 Conn_01x02, J411 Conn_01x02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

Commit message: Added comments to the schematic. Changed various component values (annotated only).
Parts:
- C401, C402, C403, C404, C405, C406, C407: symbol Device:C -> FHNW-Pro4E-FS19T8-3DPrinterBoard-STM32-rescue:C-Device
- D401, D402: symbol Device:LED -> FHNW-Pro4E-FS19T8-3DPrinterBoard-STM32-rescue:LED-Device
- D403, D404, D405: symbol Device:D_Schottky -> FHNW-Pro4E-FS19T8-3DPrinterBoard-STM32-rescue:D_Schottky-Device
- D601, D602, D603, D604, D605, D606, D607, D608: symbol Diode:BAT54S -> FHNW-Pro4E-FS19T8-3DPrinterBoard-STM32-rescue:BAT54S-Diode
- F401, F402: symbol Device:Fuse -> FHNW-Pro4E-FS19T8-3DPrinterBoard-STM32-rescue:Fuse-Device
- J401, J402, J404, J405, J407, J408, J409, J410, J411: symbol Connector_Generic:Conn_01x02 -> FHNW-Pro4E-FS19T8-3DPrinterBoard-STM32-rescue:Conn_01x02-Connector_Generic
- J403: symbol Connector:Screw_Terminal_01x04 -> FHNW-Pro4E-FS19T8-3DPrinterBoard-STM32-rescue:Screw_Terminal_01x04-Connector
- J605, J606: symbol Connector_Generic:Conn_01x03 -> FHNW-Pro4E-FS19T8-3DPrinterBoard-STM32-rescue:Conn_01x03-Connector_Generic
- R401, R402, R404, R405, R406, R407, R409, R410, R411, R413, R415, R416, R417, R418, R419, R420, R421, R422, R423: symbol Device:R -> FHNW-Pro4E-FS19T8-3DPrinterBoard-STM32-rescue:R-Device
- T401, T404, T405: symbol Transistor_FET:2N7002 -> FHNW-Pro4E-FS19T8-3DPrinterBoard-STM32-rescue:2N7002-Transistor_FET
- TH401: symbol Device:Thermistor_NTC -> FHNW-Pro4E-FS19T8-3DPrinterBoard-STM32-rescue:Thermistor_NTC-Device
Other:
- note added: "100n"
- note added: "10A"
- note added: "10k"
- note added: "10u seems way to large,\nmaybe the usual 100n?"
- note added: "3A"
- note added: "Labeled as `SERVO1` one the PCB."
- note added: "Were these resistors properly dimensioned or randomly chosen?\nR404 / R413 / R420 => 33R\nR411 / R407 => 10k"
- note added: "Why should the resistor R409 be any\ndifferent from R402 / R406 or R410?"
- note added: "Wrongly labeled as `SERVO1` as well on the PCB."
- note added: "YELLOW"
- note added: "fc = 3.545 Hz"
